File: kicad/just-40/just-40.kicad_sch (KiCad schematic)
At the start: 85 parts

Commit message: almost all routed
Parts:
- removed A1, A10, A11, A14, A15, A16, A17, A18, A19, A2, A20, A21, A22, A25, A26, A27, A28, A29, A3, A30, A31, A32, A34, A35, A36, A38, A39, A4, A5, A6, A7, A8, A9: KEY-PARTS-HS-NO-D, just-40:KEY-PARTS-HS-NO-D-1U, symbol just-40:KEY-PARTS-HS-NO-D
- removed A12: KEY-PARTS-HS-NO-D, just-40:KEY-PARTS-HS-NO-D-1.5U, symbol just-40:KEY-PARTS-HS-NO-D
- removed A13, A40: KEY-PARTS-HS-NO-D, just-40:KEY-PARTS-HS-NO-D-1.25U, symbol just-40:KEY-PARTS-HS-NO-D
- removed A23: KEY-PARTS-HS-NO-D, just-40:KEY-PARTS-HS-NO-D-2.25U, symbol just-40:KEY-PARTS-HS-NO-D
- removed A24: KEY-PARTS-HS-NO-D, just-40:KEY-PARTS-HS-NO-D-1.75U, symbol just-40:KEY-PARTS-HS-NO-D
- removed A33: KEY-PARTS-HS-NO-D, just-40:KEY-PARTS-HS-NO-D-2.75U, symbol just-40:KEY-PARTS-HS-NO-D
- removed A37: KEY-PARTS-HS-NO-D, just-40:KEY-PARTS-HS-NO-D-6.25U, symbol just-40:KEY-PARTS-HS-NO-D
- removed D1, D10, D11, D12, D13, D14, D15, D16, D17, D18, D19, D2, D20, D21, D22, D23, D24, D25, D26, D27, D28, D29, D3, D30, D31, D32, D33, D34, D35, D36, D37, D38, D39, D4, D40, D5, D6, D7, D8, D9: 1N4148, just-40:1N4148, symbol just-40:1N4148
- added A1, A10, A11, A14, A15, A16, A17, A18, A19, A2, A20, A21, A22, A25, A26, A27, A28, A29, A3, A30, A31, A32, A34, A35, A36, A38, A39, A4, A5, A6, A7, A8, A9: KEY-PARTS-HS, just-40:KEY-PARTS-HS-1U, symbol just-40:KEY-PARTS-HS
- added A12: KEY-PARTS-HS, just-40:KEY-PARTS-HS-1.5U, symbol just-40:KEY-PARTS-HS
- added A13, A40: KEY-PARTS-HS, just-40:KEY-PARTS-HS-1.25U, symbol just-40:KEY-PARTS-HS
- added A23: KEY-PARTS-HS, just-40:KEY-PARTS-HS-2.25U, symbol just-40:KEY-PARTS-HS
- added A24: KEY-PARTS-HS, just-40:KEY-PARTS-HS-1.75U, symbol just-40:KEY-PARTS-HS
- added A33: KEY-PARTS-HS, just-40:KEY-PARTS-HS-2.75U, symbol just-40:KEY-PARTS-HS
- added A37: KEY-PARTS-HS, just-40:KEY-PARTS-HS-6.25U, symbol just-40:KEY-PARTS-HS
- A41: footprint just-40:PICO-2 -> just-40:PICO-2-back
- renumbered D41 to D1, D42 to D2
Connections:
- net COL_00: now also A41.6 (GPIO4), A1.A, A13.A, A24.A, A34.A; no longer A41.14 (GPIO10)
- net COL_01: now also A41.7 (GPIO5), A14.A, A2.A, A25.A, A35.A; no longer A41.15 (GPIO11)
- net COL_02: now also A41.9 (GPIO6), A15.A, A26.A, A3.A, A36.A; no longer A41.16 (GPIO12)
- net COL_03: now also A41.10 (GPIO7), A16.A, A27.A, A4.A; no longer A41.17 (GPIO13)
- net COL_04: now also A41.11 (GPIO8), A17.A, A28.A, A5.A; no longer A41.19 (GPIO14)
- net COL_05: now also A41.14 (GPIO10), A18.A, A29.A, A37.A, A6.A; no longer A41.20 (GPIO15)
- net COL_06: now also A41.12 (GPIO9), A19.A, A30.A, A7.A; no longer A41.21 (GPIO16)
- net COL_07: now also A41.15 (GPIO11), A20.A, A31.A, A8.A; no longer A41.22 (GPIO17)
- net COL_08: now also A41.16 (GPIO12), A21.A, A32.A, A38.A, A9.A; no longer A41.24 (GPIO18)
- net COL_09: now also A41.17 (GPIO13), A10.A, A22.A, A39.A; no longer A41.25 (GPIO19)
- net COL_10: now also A41.19 (GPIO14), A11.A; no longer A41.26 (GPIO20)
- net COL_11: now also A41.20 (GPIO15), A12.A, A23.A, A33.A, A40.A; no longer A41.27 (GPIO21)
- net DIN: now also A41.31 (GPIO26_ADC0), A1.4 (DIN); no longer A41.6 (GPIO4)
- net DIN_2: now also A41.21 (GPIO16); no longer A41.9 (GPIO6)
- net D_12_13: now also A12.2 (DOUT), A13.4 (DIN)
- net D_23_24: now also A23.2 (DOUT), A24.4 (DIN)
- net D_33_34: now also A33.2 (DOUT), A34.4 (DIN)
- net GND: now also C1.1, C2.1, A1.3 (GND), A1.C_1, A10.3 (GND), A10.C_1, A11.3 (GND), A11.C_1, A12.3 (GND), A12.C_1, A13.3 (GND), A13.C_1, A14.3 (GND), A14.C_1, A15.3 (GND), A15.C_1, A16.3 (GND), A16.C_1, A17.3 (GND), A17.C_1, A18.3 (GND), A18.C_1, A19.3 (GND), A19.C_1, A2.3 (GND), A2.C_1, A20.3 (GND), A20.C_1, A21.3 (GND), A21.C_1, A22.3 (GND), A22.C_1, A23.3 (GND), A23.C_1, A24.3 (GND), A24.C_1, A25.3 (GND), A25.C_1, A26.3 (GND), A26.C_1, A27.3 (GND), A27.C_1, A28.3 (GND), A28.C_1, A29.3 (GND), A29.C_1, A3.3 (GND), A3.C_1, A30.3 (GND), A30.C_1, A31.3 (GND), A31.C_1, A32.3 (GND), A32.C_1, A33.3 (GND), A33.C_1, A34.3 (GND), A34.C_1, A35.3 (GND), A35.C_1, A36.3 (GND), A36.C_1, A37.3 (GND), A37.C_1, A38.3 (GND), A38.C_1, A39.3 (GND), A39.C_1, A4.3 (GND), A4.C_1, A40.3 (GND), A40.C_1, A5.3 (GND), A5.C_1, A6.3 (GND), A6.C_1, A7.3 (GND), A7.C_1, A8.3 (GND), A8.C_1, A9.3 (GND), A9.C_1; no longer C1.2, C2.2
- net ROW_0: now also A41.5 (GPIO3), A1.D_2, A10.D_2, A11.D_2, A12.D_2, A2.D_2, A3.D_2, A4.D_2, A5.D_2, A6.D_2, A7.D_2, A8.D_2, A9.D_2; no longer A41.1 (GPIO0)
- net ROW_1: now also A41.4 (GPIO2), A13.D_2, A14.D_2, A15.D_2, A16.D_2, A17.D_2, A18.D_2, A19.D_2, A20.D_2, A21.D_2, A22.D_2, A23.D_2; no longer A41.2 (GPIO1)
- net ROW_2: now also A41.2 (GPIO1), A24.D_2, A25.D_2, A26.D_2, A27.D_2, A28.D_2, A29.D_2, A30.D_2, A31.D_2, A32.D_2, A33.D_2; no longer A41.4 (GPIO2)
- net ROW_3: now also A41.1 (GPIO0), A34.D_2, A35.D_2, A36.D_2, A37.D_2, A38.D_2, A39.D_2, A40.D_2; no longer A41.5 (GPIO3)
- net VDD: now also C1.2, C2.2, A1.1 (VDD), A1.C_2, A10.1 (VDD), A10.C_2, A11.1 (VDD), A11.C_2, A12.1 (VDD), A12.C_2, A13.1 (VDD), A13.C_2, A14.1 (VDD), A14.C_2, A15.1 (VDD), A15.C_2, A16.1 (VDD), A16.C_2, A17.1 (VDD), A17.C_2, A18.1 (VDD), A18.C_2, A19.1 (VDD), A19.C_2, A2.1 (VDD), A2.C_2, A20.1 (VDD), A20.C_2, A21.1 (VDD), A21.C_2, A22.1 (VDD), A22.C_2, A23.1 (VDD), A23.C_2, A24.1 (VDD), A24.C_2, A25.1 (VDD), A25.C_2, A26.1 (VDD), A26.C_2, A27.1 (VDD), A27.C_2, A28.1 (VDD), A28.C_2, A29.1 (VDD), A29.C_2, A3.1 (VDD), A3.C_2, A30.1 (VDD), A30.C_2, A31.1 (VDD), A31.C_2, A32.1 (VDD), A32.C_2, A33.1 (VDD), A33.C_2, A34.1 (VDD), A34.C_2, A35.1 (VDD), A35.C_2, A36.1 (VDD), A36.C_2, A37.1 (VDD), A37.C_2, A38.1 (VDD), A38.C_2, A39.1 (VDD), A39.C_2, A4.1 (VDD), A4.C_2, A40.1 (VDD), A40.C_2, A5.1 (VDD), A5.C_2, A6.1 (VDD), A6.C_2, A7.1 (VDD), A7.C_2, A8.1 (VDD), A8.C_2, A9.1 (VDD), A9.C_2; no longer C1.1, C2.1
- new net: A20.2 (DOUT), A21.4 (DIN)
- new net: A19.2 (DOUT), A20.4 (DIN)
- new net: A20.B, A20.D_1
- new net: A22.2 (DOUT), A23.4 (DIN)
- new net: A23.B, A23.D_1
- new net: A26.2 (DOUT), A27.4 (DIN)
- new net: A25.2 (DOUT), A26.4 (DIN)
- new net: A26.B, A26.D_1
- new net: A21.2 (DOUT), A22.4 (DIN)
- new net: A21.B, A21.D_1
- new net: A39.2 (DOUT), A40.4 (DIN)
- new net: A38.2 (DOUT), A39.4 (DIN)
- new net: A39.B, A39.D_1
- new net: A32.2 (DOUT), A33.4 (DIN)
- new net: A31.2 (DOUT), A32.4 (DIN)
- new net: A32.B, A32.D_1
- new net: A10.4 (DIN), A9.2 (DOUT)
- new net: A8.2 (DOUT), A9.4 (DIN)
- new net: A9.B, A9.D_1
- new net: A11.2 (DOUT), A12.4 (DIN)
- new net: A10.2 (DOUT), A11.4 (DIN)
- new net: A11.B, A11.D_1
- new net: A28.2 (DOUT), A29.4 (DIN)
- new net: A27.2 (DOUT), A28.4 (DIN)
- new net: A28.B, A28.D_1
- new net: A2.2 (DOUT), A3.4 (DIN)
- new net: A1.2 (DOUT), A2.4 (DIN)
- new net: A2.B, A2.D_1
- new net: A30.2 (DOUT), A31.4 (DIN)
- new net: A29.2 (DOUT), A30.4 (DIN)
- new net: A30.B, A30.D_1
- new net: A22.B, A22.D_1
- new net: A7.2 (DOUT), A8.4 (DIN)
- new net: A8.B, A8.D_1
- new net: A35.2 (DOUT), A36.4 (DIN)
- new net: A34.2 (DOUT), A35.4 (DIN)
- new net: A35.B, A35.D_1
- new net: A17.2 (DOUT), A18.4 (DIN)
- new net: A16.2 (DOUT), A17.4 (DIN)
- new net: A17.B, A17.D_1
- new net: A13.2 (DOUT), A14.4 (DIN)
- new net: A13.B, A13.D_1
- new net: A18.2 (DOUT), A19.4 (DIN)
- new net: A19.B, A19.D_1
- new net: A27.B, A27.D_1
- new net: A10.B, A10.D_1
- new net: A12.B, A12.D_1
- new net: A36.2 (DOUT), A37.4 (DIN)
- new net: A36.B, A36.D_1
- new net: A37.2 (DOUT), A38.4 (DIN)
- new net: A37.B, A37.D_1
- new net: A15.2 (DOUT), A16.4 (DIN)
- new net: A14.2 (DOUT), A15.4 (DIN)
- new net: A15.B, A15.D_1
- new net: A3.2 (DOUT), A4.4 (DIN)
- new net: A3.B, A3.D_1
- new net: A34.B, A34.D_1
- new net: A14.B, A14.D_1
- new net: A24.2 (DOUT), A25.4 (DIN)
- new net: A25.B, A25.D_1
- new net: A31.B, A31.D_1
- new net: A6.2 (DOUT), A7.4 (DIN)
- new net: A5.2 (DOUT), A6.4 (DIN)
- new net: A6.B, A6.D_1
- new net: A7.B, A7.D_1
- new net: A38.B, A38.D_1
- new net: A29.B, A29.D_1
- new net: A33.B, A33.D_1
- new net: A24.B, A24.D_1
- new net: A40.B, A40.D_1
- new net: A4.2 (DOUT), A5.4 (DIN)
- new net: A5.B, A5.D_1
- new net: A1.B, A1.D_1
- new net: A4.B, A4.D_1
- new net: A18.B, A18.D_1
- new net: A16.B, A16.D_1
Other:
- moved on the sheet: C1, C2
