File: kicad/just-40/just-40.kicad_sch (KiCad schematic)
At the start: 45 parts

Commit message: pcb done - ground plate to do
Connections:
- net COL_00: now also A41.20 (GPIO15); no longer A41.6 (GPIO4)
- net COL_01: now also A41.19 (GPIO14); no longer A41.7 (GPIO5)
- net COL_02: now also A41.17 (GPIO13); no longer A41.9 (GPIO6)
- net COL_03: now also A41.16 (GPIO12); no longer A41.10 (GPIO7)
- net COL_04: now also A41.15 (GPIO11); no longer A41.11 (GPIO8)
- net COL_07: now also A41.11 (GPIO8); no longer A41.15 (GPIO11)
- net COL_08: now also A41.10 (GPIO7); no longer A41.16 (GPIO12)
- net COL_09: now also A41.9 (GPIO6); no longer A41.17 (GPIO13)
- net COL_10: now also A41.7 (GPIO5); no longer A41.19 (GPIO14)
- net COL_11: now also A41.6 (GPIO4); no longer A41.20 (GPIO15)
- net DIN: now also A41.21 (GPIO16); no longer A41.31 (GPIO26_ADC0)
- net DIN_2: now also A41.31 (GPIO26_ADC0); no longer A41.21 (GPIO16)
