File: kicad/just-40/just-40.kicad_pcb (KiCad board)
At the start: 2 copper layers, 0 parts

Commit message: wips kicad - start micropython
Parts:
- added A1: KB-SW-parts, just-40:KEY-PARTS-1U, F.Cu at (49.7, 38.0)
- added A10: KB-SW-parts, just-40:KEY-PARTS-1U, F.Cu at (263.6, 41.2)
- added A11: KB-SW-parts, just-40:KEY-PARTS-1U, F.Cu at (282.6, 41.2)
- added A12: KB-SW-parts, just-40:KEY-PARTS-1.5U, F.Cu at (306.5, 40.1)
- added A13: KB-SW-parts, just-40:KEY-PARTS-1.25U, F.Cu at (87.8, 171.8)
- added A14: KB-SW-parts, just-40:KEY-PARTS-1U, F.Cu at (28.5, 38.0)
- added A15: KB-SW-parts, just-40:KEY-PARTS-1U, F.Cu at (73.4, 32.2)
- added A16: KB-SW-parts, just-40:KEY-PARTS-1U, F.Cu at (149.8, 69.1)
- added A17: KB-SW-parts, just-40:KEY-PARTS-1U, F.Cu at (170.7, 71.0)
- added A18: KB-SW-parts, just-40:KEY-PARTS-1U, F.Cu at (193.2, 79.2)
- added A19: KB-SW-parts, just-40:KEY-PARTS-1U, F.Cu at (214.7, 78.1)
- added A2: KB-SW-parts, just-40:KEY-PARTS-1U, F.Cu at (103.6, 139.1)
- added A20: KB-SW-parts, just-40:KEY-PARTS-1U, F.Cu at (235.1, 79.2)
- added A21: KB-SW-parts, just-40:KEY-PARTS-1U, F.Cu at (256.2, 74.0)
- added A22: KB-SW-parts, just-40:KEY-PARTS-1U, F.Cu at (277.9, 79.2)
- added A23: KB-SW-parts, just-40:KEY-PARTS-2.25U, F.Cu at (308.7, 79.2)
- added A24: KB-SW-parts, just-40:KEY-PARTS-1.75U, F.Cu at (434.0, 98.8)
- added A25: KB-SW-parts, just-40:KEY-PARTS-1U, F.Cu at (366.8, 96.8)
- added A26: KB-SW-parts, just-40:KEY-PARTS-1U, F.Cu at (366.8, 116.8)
- added A27: KB-SW-parts, just-40:KEY-PARTS-1U, F.Cu at (366.8, 136.9)
- added A28: KB-SW-parts, just-40:KEY-PARTS-1U, F.Cu at (179.3, 264.0)
- added A29: KB-SW-parts, just-40:KEY-PARTS-1U, F.Cu at (179.3, 284.0)
- added A3: KB-SW-parts, just-40:KEY-PARTS-1U, F.Cu at (122.6, 139.1)
- added A30: KB-SW-parts, just-40:KEY-PARTS-1U, F.Cu at (386.8, 76.7)
- added A31: KB-SW-parts, just-40:KEY-PARTS-1U, F.Cu at (386.8, 96.8)
- added A32: KB-SW-parts, just-40:KEY-PARTS-1U, F.Cu at (386.8, 116.8)
- added A33: KB-SW-parts, just-40:KEY-PARTS-2.75U, F.Cu at (236.1, 264.0)
- added A34: KB-SW-parts, just-40:KEY-PARTS-1U, F.Cu at (386.8, 136.9)
- added A35: KB-SW-parts, just-40:KEY-PARTS-1U, F.Cu at (199.4, 264.0)
- added A36: KB-SW-parts, just-40:KEY-PARTS-1U, F.Cu at (199.4, 284.0)
- added A37: KB-SW-parts, just-40:KEY-PARTS-6.25U, F.Cu at (149.3, 223.0)
- added A38: KB-SW-parts, just-40:KEY-PARTS-1U, F.Cu at (406.9, 76.7)
- added A39: KB-SW-parts, just-40:KEY-PARTS-1U, F.Cu at (406.9, 96.8)
- added A4: KB-SW-parts, just-40:KEY-PARTS-1U, F.Cu at (141.6, 139.1)
- added A40: KB-SW-parts, just-40:KEY-PARTS-1.25U, F.Cu at (429.3, 138.9)
- added A41: PICO-2, just-40:PICO-2, F.Cu at (422.6, 228.8)
- added A5: KB-SW-parts, just-40:KEY-PARTS-1U, F.Cu at (160.6, 139.1)
- added A6: KB-SW-parts, just-40:KEY-PARTS-1U, F.Cu at (179.6, 139.1)
- added A7: KB-SW-parts, just-40:KEY-PARTS-1U, F.Cu at (198.6, 139.1)
- added A8: KB-SW-parts, just-40:KEY-PARTS-1U, F.Cu at (217.6, 139.1)
- added A9: KB-SW-parts, just-40:KEY-PARTS-1U, F.Cu at (237.2, 152.7)

Commit message: lots of wip
Parts:
- added C1: CL31A107, just-40:CL31A107, F.Cu at (84.5, 48.5)
- added C2: CL31A107, just-40:CL31A107, F.Cu at (84.5, 58.0)
- added D1: 1N4148, just-40:1N4148, F.Cu at (113.3, 47.0)
- added D10: 1N4148, just-40:1N4148, F.Cu at (235.2, 47.0)
- added D11: 1N4148, just-40:1N4148, F.Cu at (246.6, 47.0)
- added D12: 1N4148, just-40:1N4148, F.Cu at (250.4, 47.0)
- added D13: 1N4148, just-40:1N4148, F.Cu at (117.1, 50.8)
- added D14: 1N4148, just-40:1N4148, F.Cu at (132.3, 50.8)
- added D15: 1N4148, just-40:1N4148, F.Cu at (147.6, 50.8)
- added D16: 1N4148, just-40:1N4148, F.Cu at (162.8, 50.8)
- added D17: 1N4148, just-40:1N4148, F.Cu at (174.2, 50.8)
- added D18: 1N4148, just-40:1N4148, F.Cu at (185.7, 50.8)
- added D19: 1N4148, just-40:1N4148, F.Cu at (200.9, 50.8)
- added D2: 1N4148, just-40:1N4148, F.Cu at (128.5, 47.0)
- added D20: 1N4148, just-40:1N4148, F.Cu at (212.3, 50.8)
- added D21: 1N4148, just-40:1N4148, F.Cu at (223.8, 50.8)
- added D22: 1N4148, just-40:1N4148, F.Cu at (239.0, 50.8)
- added D23: 1N4148, just-40:1N4148, F.Cu at (254.2, 50.8)
- added D24: 1N4148, just-40:1N4148, F.Cu at (120.9, 54.6)
- added D25: 1N4148, just-40:1N4148, F.Cu at (136.1, 54.6)
- added D26: 1N4148, just-40:1N4148, F.Cu at (151.4, 54.6)
- added D27: 1N4148, just-40:1N4148, F.Cu at (166.6, 54.6)
- added D28: 1N4148, just-40:1N4148, F.Cu at (178.0, 54.6)
- added D29: 1N4148, just-40:1N4148, F.Cu at (189.5, 54.6)
- added D3: 1N4148, just-40:1N4148, F.Cu at (143.7, 47.0)
- added D30: 1N4148, just-40:1N4148, F.Cu at (204.7, 54.6)
- added D31: 1N4148, just-40:1N4148, F.Cu at (216.1, 54.6)
- added D32: 1N4148, just-40:1N4148, F.Cu at (227.6, 54.6)
- added D33: 1N4148, just-40:1N4148, F.Cu at (258.0, 54.6)
- added D34: 1N4148, just-40:1N4148, F.Cu at (124.7, 58.5)
- added D35: 1N4148, just-40:1N4148, F.Cu at (139.9, 58.5)
- added D36: 1N4148, just-40:1N4148, F.Cu at (155.2, 58.5)
- added D37: 1N4148, just-40:1N4148, F.Cu at (193.3, 58.5)
- added D38: 1N4148, just-40:1N4148, F.Cu at (231.4, 58.5)
- added D39: 1N4148, just-40:1N4148, F.Cu at (242.8, 58.5)
- added D4: 1N4148, just-40:1N4148, F.Cu at (159.0, 47.0)
- added D40: 1N4148, just-40:1N4148, F.Cu at (261.9, 58.5)
- added D41: SK6812MINI-E, just-40:SK6812MINI-E, F.Cu at (92.0, 58.0)
- added D42: SK6812MINI-E, just-40:SK6812MINI-E, F.Cu at (92.0, 48.5)
- added D5: 1N4148, just-40:1N4148, F.Cu at (170.4, 47.0)
- added D6: 1N4148, just-40:1N4148, F.Cu at (181.8, 47.0)
- added D7: 1N4148, just-40:1N4148, F.Cu at (197.1, 47.0)
- added D8: 1N4148, just-40:1N4148, F.Cu at (208.5, 47.0)
- added D9: 1N4148, just-40:1N4148, F.Cu at (219.9, 47.0)
- added REF**: Mount-Hole, just-40:Mount-Hole, F.Cu at (49.0, 73.5)
- added REF**: Mount-Hole, just-40:Mount-Hole, F.Cu at (38.0, 53.0)
- added REF**: Mount-Hole, just-40:Mount-Hole, F.Cu at (107.5, 44.0)
- added REF**: Mount-Hole, just-40:Mount-Hole, F.Cu at (266.5, 62.0)
- added REF**: Mount-Hole, just-40:Mount-Hole, F.Cu at (73.0, 53.0)
- added REF**: Mount-Hole, just-40:Mount-Hole, F.Cu at (107.5, 62.0)
- added REF**: Mount-Hole, just-40:Mount-Hole, F.Cu at (246.0, 130.0)
- added REF**: Mount-Hole, just-40:Mount-Hole, F.Cu at (144.0, 73.5)
- added REF**: Mount-Hole, just-40:Mount-Hole, F.Cu at (243.5, 73.5)
- added REF**: Mount-Hole, just-40:Mount-Hole, F.Cu at (136.5, 130.5)
- added REF**: Mount-Hole, just-40:Mount-Hole, F.Cu at (266.5, 44.0)
- added REF**: Mount-Hole, just-40:Mount-Hole, F.Cu at (49.0, 130.5)
- A1, A10, A11, A14, A15, A16, A17, A18, A19, A2, A20, A21, A22, A25, A26, A27, A28, A29, A3, A30, A31, A32, A34, A35, A36, A38, A39, A4, A5, A6, A7, A8, A9: value KB-SW-parts -> KEY-PARTS-HS-NO-D; footprint just-40:KEY-PARTS-1U -> just-40:KEY-PARTS-HS-NO-D-1U
- A12: value KB-SW-parts -> KEY-PARTS-HS-NO-D; footprint just-40:KEY-PARTS-1.5U -> just-40:KEY-PARTS-HS-NO-D-1.5U
- A13, A40: value KB-SW-parts -> KEY-PARTS-HS-NO-D; footprint just-40:KEY-PARTS-1.25U -> just-40:KEY-PARTS-HS-NO-D-1.25U
- A23: value KB-SW-parts -> KEY-PARTS-HS-NO-D; footprint just-40:KEY-PARTS-2.25U -> just-40:KEY-PARTS-HS-NO-D-2.25U
- A24: value KB-SW-parts -> KEY-PARTS-HS-NO-D; footprint just-40:KEY-PARTS-1.75U -> just-40:KEY-PARTS-HS-NO-D-1.75U
- A33: value KB-SW-parts -> KEY-PARTS-HS-NO-D; footprint just-40:KEY-PARTS-2.75U -> just-40:KEY-PARTS-HS-NO-D-2.75U
- A37: value KB-SW-parts -> KEY-PARTS-HS-NO-D; footprint just-40:KEY-PARTS-6.25U -> just-40:KEY-PARTS-HS-NO-D-6.25U
- moved A41 407.0 mm to (55.5, 53.0)
- moved A24 387.6 mm to (46.6, 111.5)
- moved A34 347.4 mm to (39.5, 130.5)
- moved A25 294.4 mm to (72.8, 111.5)
- moved A26 275.1 mm to (91.8, 111.5)
- moved A27 257.3 mm to (110.8, 111.5)
- moved A30 221.8 mm to (167.8, 111.5)
- moved A31 200.6 mm to (186.8, 111.5)
- moved A38 199.0 mm to (215.2, 130.5)
- moved A36 196.0 mm to (77.5, 130.5)
- moved A35 194.1 mm to (58.5, 130.5)
- moved A32 181.1 mm to (205.8, 111.5)
- moved A39 175.9 mm to (234.2, 130.5)
- moved A29 175.2 mm to (148.8, 111.5)
- moved A40 173.9 mm to (255.6, 130.5)
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Connections:
- A1 pad 1: +5V -> VDD
- A1 pad B: Net-(A1-PadB) -> Net-(D1-A)
- A1 pad C_2: +5V -> VDD
- A10 pad 1: +5V -> VDD
- A10 pad B: Net-(A10-PadB) -> Net-(D10-A)
- A10 pad C_2: +5V -> VDD
- A11 pad 1: +5V -> VDD
- A11 pad B: Net-(A11-PadB) -> Net-(D11-A)
- A11 pad C_2: +5V -> VDD
- A12 pad 1: +5V -> VDD
- A12 pad B: Net-(A12-PadB) -> Net-(D12-A)
- A12 pad C_2: +5V -> VDD
- A13 pad 1: +5V -> VDD
- A13 pad B: Net-(A13-PadB) -> Net-(D13-A)
- A13 pad C_2: +5V -> VDD
- A14 pad 1: +5V -> VDD
- A14 pad B: Net-(A14-PadB) -> Net-(D14-A)
- A14 pad C_2: +5V -> VDD
- A15 pad 1: +5V -> VDD
- A15 pad B: Net-(A15-PadB) -> Net-(D15-A)
- A15 pad C_2: +5V -> VDD
- A16 pad 1: +5V -> VDD
- A16 pad B: Net-(A16-PadB) -> Net-(D16-A)
- A16 pad C_2: +5V -> VDD
- A17 pad 1: +5V -> VDD
- A17 pad B: Net-(A17-PadB) -> Net-(D17-A)
- A17 pad C_2: +5V -> VDD
- A18 pad 1: +5V -> VDD
- A18 pad B: Net-(A18-PadB) -> Net-(D18-A)
- A18 pad C_2: +5V -> VDD
- A19 pad 1: +5V -> VDD
- A19 pad B: Net-(A19-PadB) -> Net-(D19-A)
- A19 pad C_2: +5V -> VDD
- A2 pad 1: +5V -> VDD
- A2 pad B: Net-(A2-PadB) -> Net-(D2-A)
- A2 pad C_2: +5V -> VDD
- A20 pad 1: +5V -> VDD
- A20 pad B: Net-(A20-PadB) -> Net-(D20-A)
- A20 pad C_2: +5V -> VDD
- A21 pad 1: +5V -> VDD
- A21 pad B: Net-(A21-PadB) -> Net-(D21-A)
- A21 pad C_2: +5V -> VDD
- A22 pad 1: +5V -> VDD
- A22 pad B: Net-(A22-PadB) -> Net-(D22-A)
- A22 pad C_2: +5V -> VDD
- A23 pad 1: +5V -> VDD
- A23 pad B: Net-(A23-PadB) -> Net-(D23-A)
- A23 pad C_2: +5V -> VDD
- A24 pad 1: +5V -> VDD
- A24 pad B: Net-(A24-PadB) -> Net-(D24-A)
- A24 pad C_2: +5V -> VDD
- A25 pad 1: +5V -> VDD
- A25 pad B: Net-(A25-PadB) -> Net-(D25-A)
- A25 pad C_2: +5V -> VDD
- A26 pad 1: +5V -> VDD
- A26 pad B: Net-(A26-PadB) -> Net-(D26-A)
- A26 pad C_2: +5V -> VDD
- A27 pad 1: +5V -> VDD
- A27 pad B: Net-(A27-PadB) -> Net-(D27-A)
- A27 pad C_2: +5V -> VDD
- A28 pad 1: +5V -> VDD
- A28 pad B: Net-(A28-PadB) -> Net-(D28-A)
- A28 pad C_2: +5V -> VDD
- A29 pad 1: +5V -> VDD
- A29 pad B: Net-(A29-PadB) -> Net-(D29-A)
- A29 pad C_2: +5V -> VDD
- A3 pad 1: +5V -> VDD
- A3 pad B: Net-(A3-PadB) -> Net-(D3-A)
- A3 pad C_2: +5V -> VDD
- A30 pad 1: +5V -> VDD
- A30 pad B: Net-(A30-PadB) -> Net-(D30-A)
- A30 pad C_2: +5V -> VDD
- A31 pad 1: +5V -> VDD
- A31 pad B: Net-(A31-PadB) -> Net-(D31-A)
- A31 pad C_2: +5V -> VDD
- A32 pad 1: +5V -> VDD
- A32 pad B: Net-(A32-PadB) -> Net-(D32-A)
- A32 pad C_2: +5V -> VDD
- A33 pad 1: +5V -> VDD
- A33 pad B: Net-(A33-PadB) -> Net-(D33-A)
- A33 pad C_2: +5V -> VDD
- A34 pad 1: +5V -> VDD
- A34 pad B: Net-(A34-PadB) -> Net-(D34-A)
- A34 pad C_2: +5V -> VDD
- A35 pad 1: +5V -> VDD
- A35 pad B: Net-(A35-PadB) -> Net-(D35-A)
- A35 pad C_2: +5V -> VDD
- A36 pad 1: +5V -> VDD
- A36 pad B: Net-(A36-PadB) -> Net-(D36-A)
- A36 pad C_2: +5V -> VDD
- A37 pad 1: +5V -> VDD
- A37 pad B: Net-(A37-PadB) -> Net-(D37-A)
- A37 pad C_2: +5V -> VDD
- A38 pad 1: +5V -> VDD
- A38 pad B: Net-(A38-PadB) -> Net-(D38-A)
- A38 pad C_2: +5V -> VDD
- A39 pad 1: +5V -> VDD
- A39 pad B: Net-(A39-PadB) -> Net-(D39-A)
- A39 pad C_2: +5V -> VDD
- A4 pad 1: +5V -> VDD
- A4 pad B: Net-(A4-PadB) -> Net-(D4-A)
- A4 pad C_2: +5V -> VDD
- A40 pad 1: +5V -> VDD
- A40 pad 2: DOUT -> unconnected-(A40-DOUT-Pad2)
- A40 pad B: Net-(A40-PadB) -> Net-(D40-A)
- A40 pad C_2: +5V -> VDD
- A41 pad 36: unconnected-(A41-3V3-Pad36) -> VDD
- A41 pad 6: unconnected-(A41-GPIO4-Pad6) -> DIN
- A41 pad 9: unconnected-(A41-GPIO6-Pad9) -> DIN_2
- A5 pad 1: +5V -> VDD
- A5 pad B: Net-(A5-PadB) -> Net-(D5-A)
- A5 pad C_2: +5V -> VDD
- A6 pad 1: +5V -> VDD
- A6 pad B: Net-(A6-PadB) -> Net-(D6-A)
- A6 pad C_2: +5V -> VDD
- A7 pad 1: +5V -> VDD
- A7 pad B: Net-(A7-PadB) -> Net-(D7-A)
- A7 pad C_2: +5V -> VDD
- A8 pad 1: +5V -> VDD
- A8 pad B: Net-(A8-PadB) -> Net-(D8-A)
- A8 pad C_2: +5V -> VDD
- A9 pad 1: +5V -> VDD
- A9 pad B: Net-(A9-PadB) -> Net-(D9-A)
- A9 pad C_2: +5V -> VDD
Routing:
- net VDD: track 0.00 -> 457.3 mm
- net D_12_13: track 0.00 -> 246.7 mm
- net D_33_34: track 0.00 -> 237.3 mm
- net D_23_24: track 0.00 -> 235.2 mm
- net GND: track 0.00 -> 194.4 mm
- net Net-(D34-A): track 0.00 -> 171.9 mm, vias 0 -> 3
- net Net-(D24-A): track 0.00 -> 137.6 mm, vias 0 -> 3
- net ROW_3: track 0.00 -> 137.2 mm
- net ROW_2: track 0.00 -> 137.2 mm
- net ROW_1: track 0.00 -> 137.2 mm
- net ROW_0: track 0.00 -> 137.2 mm
- net Net-(D25-A): track 0.00 -> 126.9 mm, vias 0 -> 3
- net Net-(D27-A): track 0.00 -> 112.9 mm, vias 0 -> 3
- net Net-(D13-A): track 0.00 -> 105.8 mm, vias 0 -> 3
- net Net-(D14-A): track 0.00 -> 102.4 mm, vias 0 -> 3
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Other:
- board outline added: 239.5 x 98 mm
- board text added: "Caps"
- board text added: "Nums"

Commit message: almost all routed
Parts:
- removed D10, D11, D12, D13, D14, D15, D16, D17, D18, D19, D20, D21, D22, D23, D24, D25, D26, D27, D28, D29, D3, D30, D31, D32, D33, D34, D35, D36, D37, D38, D39, D4, D40, D5, D6, D7, D8, D9: 1N4148, just-40:1N4148
- removed D41, D42: SK6812MINI-E, just-40:SK6812MINI-E
- removed the REF** at (49.0, 73.5)
- removed the REF** at (38.0, 53.0)
- removed the REF** at (107.5, 44.0)
- removed the REF** at (266.5, 62.0)
- removed the REF** at (73.0, 53.0)
- removed the REF** at (107.5, 62.0)
- removed the REF** at (246.0, 130.0)
- removed the REF** at (144.0, 73.5)
- removed the REF** at (243.5, 73.5)
- removed the REF** at (136.5, 130.5)
- removed the REF** at (266.5, 44.0)
- removed the REF** at (49.0, 130.5)
- added REF**: Mount-Hole, just-40:Mount-Hole, F.Cu at (104.0, 58.0)
- added REF**: Mount-Hole, just-40:Mount-Hole, F.Cu at (265.5, 58.0)
- added REF**: Mount-Hole, just-40:Mount-Hole, F.Cu at (186.5, 132.0)
- added REF**: Mount-Hole, just-40:Mount-Hole, F.Cu at (28.0, 58.0)
- added REF**: Mount-Hole, just-40:Mount-Hole, F.Cu at (180.0, 58.0)
- added REF**: Mount-Hole, just-40:Mount-Hole, F.Cu at (108.0, 132.0)
- added REF**: Mount-Hole, just-40:Mount-Hole, F.Cu at (28.0, 95.0)
- added REF**: Mount-Hole, just-40:Mount-Hole, F.Cu at (108.8, 95.0)
- added REF**: Mount-Hole, just-40:Mount-Hole, F.Cu at (184.8, 95.0)
- added REF**: Mount-Hole, just-40:Mount-Hole, F.Cu at (28.0, 132.0)
- added REF**: Mount-Hole, just-40:Mount-Hole, F.Cu at (265.5, 132.0)
- added REF**: Mount-Hole, just-40:Mount-Hole, F.Cu at (265.5, 95.0)
- A1, A10, A11, A14, A15, A16, A17, A18, A19, A2, A20, A21, A22, A25, A26, A27, A28, A29, A3, A30, A31, A32, A34, A35, A36, A38, A39, A4, A5, A6, A7, A8, A9: value KEY-PARTS-HS-NO-D -> KEY-PARTS-HS; footprint just-40:KEY-PARTS-HS-NO-D-1U -> just-40:KEY-PARTS-HS-1U
- A12: value KEY-PARTS-HS-NO-D -> KEY-PARTS-HS; footprint just-40:KEY-PARTS-HS-NO-D-1.5U -> just-40:KEY-PARTS-HS-1.5U
- A13, A40: value KEY-PARTS-HS-NO-D -> KEY-PARTS-HS; footprint just-40:KEY-PARTS-HS-NO-D-1.25U -> just-40:KEY-PARTS-HS-1.25U
- A23: value KEY-PARTS-HS-NO-D -> KEY-PARTS-HS; footprint just-40:KEY-PARTS-HS-NO-D-2.25U -> just-40:KEY-PARTS-HS-2.25U
- A24: value KEY-PARTS-HS-NO-D -> KEY-PARTS-HS; footprint just-40:KEY-PARTS-HS-NO-D-1.75U -> just-40:KEY-PARTS-HS-1.75U
- A33: value KEY-PARTS-HS-NO-D -> KEY-PARTS-HS; footprint just-40:KEY-PARTS-HS-NO-D-2.75U -> just-40:KEY-PARTS-HS-2.75U
- A37: value KEY-PARTS-HS-NO-D -> KEY-PARTS-HS; footprint just-40:KEY-PARTS-HS-NO-D-6.25U -> just-40:KEY-PARTS-HS-6.25U
- A41: footprint just-40:PICO-2 -> just-40:PICO-2-back
- D1, D2: value 1N4148 -> SK6812MINI-E; footprint just-40:1N4148 -> just-40:SK6812MINI-E
- moved C1 177.2 mm to (259.0, 79.1), turned to 0 degrees
- moved C2 177.2 mm to (259.0, 88.4), turned to 0 degrees
- moved D1 156.3 mm to (264.0, 88.4), turned to 90 degrees
- moved D2 139.3 mm to (264.0, 79.1), turned to 90 degrees
- moved A41 14.5 mm to (55.5, 67.5)
- moved A1 6.32 mm to (37.5, 67.5)
- moved A10 6.32 mm to (208.5, 67.5)
- moved A11 6.32 mm to (227.5, 67.5)
- moved A12 6.32 mm to (251.2, 67.5)
- moved A13 6.32 mm to (39.9, 86.5)
- moved A14 6.32 mm to (61.2, 86.5)
- moved A15 6.32 mm to (80.2, 86.5)
- moved A16 6.32 mm to (99.2, 86.5)
- moved A17 6.32 mm to (118.2, 86.5)
- moved A18 6.32 mm to (137.2, 86.5)
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Connections:
- A1 pad B: Net-(D1-A) -> Net-(A1-PadB)
- A10 pad B: Net-(D10-A) -> Net-(A10-PadB)
- A11 pad B: Net-(D11-A) -> Net-(A11-PadB)
- A12 pad B: Net-(D12-A) -> Net-(A12-PadB)
- A13 pad B: Net-(D13-A) -> Net-(A13-PadB)
- A14 pad B: Net-(D14-A) -> Net-(A14-PadB)
- A15 pad B: Net-(D15-A) -> Net-(A15-PadB)
- A16 pad B: Net-(D16-A) -> Net-(A16-PadB)
- A17 pad B: Net-(D17-A) -> Net-(A17-PadB)
- A18 pad B: Net-(D18-A) -> Net-(A18-PadB)
- A19 pad B: Net-(D19-A) -> Net-(A19-PadB)
- A2 pad B: Net-(D2-A) -> Net-(A2-PadB)
- A20 pad B: Net-(D20-A) -> Net-(A20-PadB)
- A21 pad B: Net-(D21-A) -> Net-(A21-PadB)
- A22 pad B: Net-(D22-A) -> Net-(A22-PadB)
- A23 pad B: Net-(D23-A) -> Net-(A23-PadB)
- A24 pad B: Net-(D24-A) -> Net-(A24-PadB)
- A25 pad B: Net-(D25-A) -> Net-(A25-PadB)
- A26 pad B: Net-(D26-A) -> Net-(A26-PadB)
- A27 pad B: Net-(D27-A) -> Net-(A27-PadB)
- A28 pad B: Net-(D28-A) -> Net-(A28-PadB)
- A29 pad B: Net-(D29-A) -> Net-(A29-PadB)
- A3 pad B: Net-(D3-A) -> Net-(A3-PadB)
- A30 pad B: Net-(D30-A) -> Net-(A30-PadB)
- A31 pad B: Net-(D31-A) -> Net-(A31-PadB)
- A32 pad B: Net-(D32-A) -> Net-(A32-PadB)
- A33 pad B: Net-(D33-A) -> Net-(A33-PadB)
- A34 pad B: Net-(D34-A) -> Net-(A34-PadB)
- A35 pad B: Net-(D35-A) -> Net-(A35-PadB)
- A36 pad B: Net-(D36-A) -> Net-(A36-PadB)
- A37 pad B: Net-(D37-A) -> Net-(A37-PadB)
- A38 pad B: Net-(D38-A) -> Net-(A38-PadB)
- A39 pad B: Net-(D39-A) -> Net-(A39-PadB)
- A4 pad B: Net-(D4-A) -> Net-(A4-PadB)
- A40 pad B: Net-(D40-A) -> Net-(A40-PadB)
- A41 pad 1: ROW_0 -> ROW_3
- A41 pad 10: unconnected-(A41-GPIO7-Pad10) -> COL_03
- A41 pad 11: unconnected-(A41-GPIO8-Pad11) -> COL_04
- A41 pad 12: unconnected-(A41-GPIO9-Pad12) -> COL_06
- A41 pad 14: COL_00 -> COL_05
- A41 pad 15: COL_01 -> COL_07
- A41 pad 16: COL_02 -> COL_08
- A41 pad 17: COL_03 -> COL_09
- A41 pad 19: COL_04 -> COL_10
- A41 pad 2: ROW_1 -> ROW_2
- A41 pad 20: COL_05 -> COL_11
- A41 pad 21: COL_06 -> DIN_2
- A41 pad 22: COL_07 -> unconnected-(A41-GPIO17-Pad22)
- A41 pad 24: COL_08 -> unconnected-(A41-GPIO18-Pad24)
- A41 pad 25: COL_09 -> unconnected-(A41-GPIO19-Pad25)
- A41 pad 26: COL_10 -> unconnected-(A41-GPIO20-Pad26)
- A41 pad 27: COL_11 -> unconnected-(A41-GPIO21-Pad27)
- A41 pad 31: unconnected-(A41-GPIO26_ADC0-Pad31) -> DIN
- A41 pad 4: ROW_2 -> ROW_1
- A41 pad 5: ROW_3 -> ROW_0
- A41 pad 6: DIN -> COL_00
- A41 pad 7: unconnected-(A41-GPIO5-Pad7) -> COL_01
- A41 pad 9: DIN_2 -> COL_02
- A5 pad B: Net-(D5-A) -> Net-(A5-PadB)
- A6 pad B: Net-(D6-A) -> Net-(A6-PadB)
- A7 pad B: Net-(D7-A) -> Net-(A7-PadB)
- A8 pad B: Net-(D8-A) -> Net-(A8-PadB)
- A9 pad B: Net-(D9-A) -> Net-(A9-PadB)
- C1 pad 1: VDD -> GND
- C1 pad 2: GND -> VDD
- C2 pad 1: VDD -> GND
- C2 pad 2: GND -> VDD
- D1 pad 1: ROW_0 -> VDD
- D1 pad 2: Net-(D1-A) -> Net-(D1-DOUT)
- D2 pad 1: ROW_0 -> VDD
- D2 pad 2: Net-(D2-A) -> unconnected-(D2-DOUT-Pad2)
Routing:
- net VDD: track 457.3 -> 1057.7 mm, vias 0 -> 4
- net GND: track 194.4 -> 664.1 mm, vias 0 -> 24
- net DIN_2: track 0.00 -> 197.6 mm, vias 0 -> 2
- net COL_11: track 77.8 -> 258.6 mm, vias 4 -> 5
- net Net-(D34-A): track 171.9 -> 0.00 mm, vias 3 -> 0
- net ROW_3: track 137.2 -> 305.7 mm, vias 0 -> 1
- net COL_10: track 2.52 -> 162.0 mm, vias 1 -> 2
- net COL_09: track 74.4 -> 218.4 mm, vias 3 -> 4
- net ROW_2: track 137.2 -> 276.7 mm, vias 0 -> 1
- net Net-(D24-A): track 137.6 -> 0.00 mm, vias 3 -> 0
- net ROW_1: track 137.2 -> 271.0 mm, vias 0 -> 1
- net COL_08: track 76.6 -> 204.6 mm, vias 4 -> 5
- net Net-(D25-A): track 126.9 -> 0.00 mm, vias 3 -> 0
- net Net-(D27-A): track 112.9 -> 0.00 mm, vias 3 -> 0
- net COL_07: track 51.5 -> 160.8 mm, vias 3 -> 4
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Other:
- board size 239.5 x 98 mm -> 241.5 x 78 mm
- board text removed: "Caps"
- board text removed: "Nums"

Commit message: pcb done - ground plate to do
Parts:
- added REF**: Mount-Hole, just-40:Mount-Hole, F.Cu at (265.5, 77.0)
- added REF**: Mount-Hole, just-40:Mount-Hole, F.Cu at (108.8, 77.0)
- added REF**: Mount-Hole, just-40:Mount-Hole, F.Cu at (265.5, 81.0)
- added REF**: Mount-Hole, just-40:Mount-Hole, F.Cu at (108.8, 81.0)
- moved A41 182.6 mm to (238.1, 67.5)
- moved REF** 157.4 mm to (28.0, 81.0)
- moved REF** 82.0 mm to (184.8, 81.0)
- moved REF** 78.1 mm to (184.8, 77.0)
- moved REF** 18.0 mm to (28.0, 77.0)
- moved C1 16.9 mm to (259.0, 96.0)
- moved D2 16.9 mm to (264.0, 96.0)
- moved C2 1.89 mm to (259.0, 86.5)
- moved D1 1.89 mm to (264.0, 86.5)
Connections:
- A41 pad 10: COL_03 -> COL_08
- A41 pad 11: COL_04 -> COL_07
- A41 pad 15: COL_07 -> COL_04
- A41 pad 16: COL_08 -> COL_03
- A41 pad 17: COL_09 -> COL_02
- A41 pad 19: COL_10 -> COL_01
- A41 pad 20: COL_11 -> COL_00
- A41 pad 21: DIN_2 -> DIN
- A41 pad 31: DIN -> DIN_2
- A41 pad 6: COL_00 -> COL_11
- A41 pad 7: COL_01 -> COL_10
- A41 pad 9: COL_02 -> COL_09
Routing:
- net GND: track 664.1 -> 1115.1 mm, vias 24 -> 0
- net COL_00: track 90.9 -> 284.2 mm, vias 4 -> 6
- net COL_11: track 258.6 -> 84.7 mm, vias 5 -> 3
- net DIN: track 41.9 -> 193.1 mm
- net DIN_2: track 197.6 -> 46.8 mm, vias 2 -> 1
- net COL_01: track 92.0 -> 242.3 mm, vias 4 -> 6
- net COL_10: track 162.0 -> 34.0 mm, vias 2 -> 0
- net COL_02: track 103.8 -> 226.8 mm, vias 4 -> 6
- net COL_09: track 218.4 -> 107.4 mm
- net COL_03: track 90.4 -> 183.6 mm, vias 3 -> 5
- net COL_08: track 204.6 -> 126.4 mm
- net COL_04: track 102.0 -> 167.5 mm, vias 3 -> 5
- net COL_07: track 160.8 -> 117.7 mm
- net VDD: track 1057.7 -> 1090.2 mm, vias 4 -> 2
- net COL_05: track 140.3 -> 172.6 mm, vias 4 -> 6
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
Commit message: pcb ground plane done - add 3d images
Routing:
- net DIN: track 193.1 -> 194.7 mm
- net COL_00: track 284.2 -> 285.6 mm
- net D_12_13: track 247.5 -> 248.7 mm
- added copper zone on B.Cu, net GND
