File: kicad/just-40/just-40.kicad_pcb (KiCad board)
At the start: 2 copper layers, 241.5 x 78 mm, 61 parts

Commit message: gerber ready
Parts:
- removed C1, C2: CL31A107, just-40:CL31A107
- removed D1, D2: SK6812MINI-E, just-40:SK6812MINI-E
- removed REF** (x16): Mount-Hole, just-40:Mount-Hole
- added H1: RP2350-Tyny-USB, just-40:RP2350-Tiny-USB, F.Cu at (254.5, 72.5)
- added H2: mount-hole, just-40:Mount-Hole, F.Cu at (26.0, 26.0)
- added H3: mount-hole, just-40:Mount-Hole, F.Cu at (101.0, 26.0)
- added H4: mount-hole, just-40:Mount-Hole, F.Cu at (177.0, 26.0)
- added H5: mount-hole, just-40:Mount-Hole, F.Cu at (261.5, 26.0)
- added H6: mount-hole, just-40:Mount-Hole, F.Cu at (26.0, 100.0)
- added H7: mount-hole, just-40:Mount-Hole, F.Cu at (102.0, 100.0)
- added H8: mount-hole, just-40:Mount-Hole, F.Cu at (185.5, 100.0)
- added H9: mount-hole, just-40:Mount-Hole, F.Cu at (261.5, 100.0)
- A34: footprint just-40:KEY-PARTS-HS-1U -> just-40:KEY-PARTS-HS-1.25U
- A40: footprint just-40:KEY-PARTS-HS-1.25U -> just-40:KEY-PARTS-HS-1U
- A41: value PICO-2 -> RP2350-Tiny; footprint just-40:PICO-2-back -> just-40:RP2350-Tiny
- moved A41 70.5 mm to (171.5, 90.5), turned to 180 degrees
- moved A1 33.1 mm to (34.5, 34.5)
- moved A10 33.1 mm to (205.5, 34.5)
- moved A11 33.1 mm to (224.5, 34.5)
- moved A12 33.1 mm to (248.2, 34.5)
- moved A13 33.1 mm to (36.9, 53.5)
- moved A14 33.1 mm to (58.2, 53.5)
- moved A15 33.1 mm to (77.2, 53.5)
- moved A16 33.1 mm to (96.2, 53.5)
- moved A17 33.1 mm to (115.2, 53.5)
- moved A18 33.1 mm to (134.2, 53.5)
- moved A19 33.1 mm to (153.2, 53.5)
- moved A2 33.1 mm to (53.5, 34.5)
- moved A20 33.1 mm to (172.2, 53.5)
- moved A21 33.1 mm to (191.2, 53.5)
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Connections:
- A41 pad 1: ROW_3 -> COL_10
- A41 pad 10: COL_08 -> COL_01
- A41 pad 11: COL_07 -> COL_00
- A41 pad 12: COL_06 -> DIN
- A41 pad 13: GND -> unconnected-(A41-GPIO13-Pad13)
- A41 pad 14: COL_05 -> ROW_3
- A41 pad 15: COL_04 -> ROW_2
- A41 pad 2: ROW_2 -> COL_11
- A41 pad 26: unconnected-(A41-GPIO20-Pad26) -> ROW_1
- A41 pad 27: unconnected-(A41-GPIO21-Pad27) -> ROW_0
- A41 pad 28: GND -> unconnected-(A41-GPIO28_ADC2-Pad28)
- A41 pad 3: GND -> COL_08
- A41 pad 4: ROW_1 -> COL_07
- A41 pad 5: ROW_0 -> COL_06
- A41 pad 6: COL_11 -> COL_03
- A41 pad 7: COL_10 -> COL_05
- A41 pad 8: GND -> COL_04
- A41 pad 9: COL_09 -> COL_02
Routing:
- net COL_10: track 34.0 -> 122.5 mm, vias 0 -> 2
- net COL_00: track 285.6 -> 199.9 mm, vias 6 -> 4
- net COL_05: track 172.6 -> 95.1 mm
- net COL_04: track 167.5 -> 90.4 mm, vias 5 -> 4
- net COL_02: track 226.8 -> 152.0 mm
- net COL_06: track 133.9 -> 60.1 mm
- net VDD: track 1090.2 -> 1020.2 mm, vias 2 -> 8
- net COL_01: track 242.3 -> 173.7 mm, vias 6 -> 5
- net ROW_0: track 261.4 -> 329.3 mm, vias 0 -> 2
- net COL_07: track 117.7 -> 49.9 mm
- net COL_03: track 183.6 -> 116.0 mm, vias 5 -> 4
- net COL_11: track 84.7 -> 149.7 mm, vias 3 -> 6
- net DIN_2: track 46.8 -> 0.00 mm, vias 1 -> 0
- net ROW_1: track 252.4 -> 298.6 mm, vias 1 -> 2
- net ROW_3: track 292.5 -> 253.7 mm, vias 1 -> 2
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Other:
- board size 241.5 x 78 mm -> 239.5 x 78 mm

Commit message: wips
Parts:
- added G***: LOGO, just-40:great-wave-50, B.Cu at (147.2, 214.0)
- added H10: mount-hole, just-40:Mount-Hole, F.Cu at (104.5, 177.0)
- added H11: mount-hole, just-40:Mount-Hole, F.Cu at (180.5, 177.0)
- added H12: mount-hole, just-40:Mount-Hole, F.Cu at (265.0, 177.0)
- added H13: mount-hole, just-40:Mount-Hole, F.Cu at (29.5, 251.0)
- added H14: mount-hole, just-40:Mount-Hole, F.Cu at (104.5, 251.0)
- added H15: mount-hole, just-40:Mount-Hole, F.Cu at (180.5, 251.0)
- added H16: mount-hole, just-40:Mount-Hole, F.Cu at (265.0, 251.0)
- A1, A10, A11, A14, A15, A16, A17, A18, A19, A2, A20, A21, A22, A25, A26, A27, A28, A29, A3, A30, A31, A32, A35, A36, A38, A39, A4, A5, A6, A7, A8, A9: footprint just-40:KEY-PARTS-HS-1U -> just-40:SW-LED-D-center-1U
- A12: footprint just-40:KEY-PARTS-HS-1.5U -> just-40:SW-LED-D-center-1.5U
- A13: footprint just-40:KEY-PARTS-HS-1.25U -> just-40:SW-LED-D-center-1.25U
- A23: footprint just-40:KEY-PARTS-HS-2.25U -> just-40:SW-LED-D-center-2.25U
- A24: footprint just-40:KEY-PARTS-HS-1.75U -> just-40:SW-LED-D-center-1.75U
- A33: footprint just-40:KEY-PARTS-HS-2.75U -> just-40:SW-LED-D-center-2.75U
- A34: footprint just-40:KEY-PARTS-HS-1.25U -> just-40:SW-LED-D-center-1U
- A37: footprint just-40:KEY-PARTS-HS-6.25U -> just-40:SW-LED-D-center-6.25U
- A40: footprint just-40:KEY-PARTS-HS-1U -> just-40:SW-LED-D-center-1.25U
- H1: value RP2350-Tyny-USB -> mount-hole; footprint just-40:RP2350-Tiny-USB -> just-40:Mount-Hole
- H9: value mount-hole -> RP2350-Tiny-USB; footprint just-40:Mount-Hole -> just-40:RP2350-Tiny-USB
- moved H5 259.2 mm to (29.5, 141.5)
- moved H9 240.2 mm to (36.5, 184.0)
- moved H1 225.1 mm to (29.5, 67.5)
- moved H4 97.3 mm to (265.0, 67.5)
- moved H3 89.7 mm to (180.5, 67.5)
- moved H8 89.7 mm to (265.0, 141.5)
- moved H2 88.8 mm to (104.5, 67.5)
- moved H6 88.8 mm to (104.5, 141.5)
- moved H7 88.8 mm to (180.5, 141.5)
- moved A41 66.0 mm to (121.0, 133.0), turned to 0 degrees
- moved A1 41.6 mm to (38.0, 76.0)
- moved A10 41.6 mm to (209.0, 76.0)
- moved A11 41.6 mm to (228.0, 76.0)
- moved A12 41.6 mm to (251.8, 76.0)
- moved A13 41.6 mm to (40.4, 95.0)
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Connections:
- net D_12_13 renamed Net-(A12-DOUT)
- net D_23_24 renamed Net-(A23-DOUT)
- net D_33_34 renamed Net-(A33-DOUT)
- net VDD renamed V_LED
- A11 pad A: COL_10 -> COL_09
- A11 pad D_2: ROW_0 -> ROW_2
- A12 pad A: COL_11 -> COL_10
- A23 pad A: COL_11 -> COL_10
- A33 pad A: COL_11 -> COL_10
- A40 pad A: COL_11 -> COL_10
- A41 pad 0: COL_09 -> DIN
- A41 pad 1: COL_10 -> COL_00
- A41 pad 10: COL_01 -> COL_07
- A41 pad 11: COL_00 -> COL_08
- A41 pad 12: DIN -> COL_09
- A41 pad 13: unconnected-(A41-GPIO13-Pad13) -> COL_05
- A41 pad 14: ROW_3 -> COL_10
- A41 pad 15: ROW_2 -> ROW_3
- A41 pad 2: COL_11 -> COL_01
- A41 pad 26: ROW_1 -> unconnected-(A41-GPIO26_ADC0-Pad26)
- A41 pad 27: ROW_0 -> unconnected-(A41-GPIO27_ADC1-Pad27)
- A41 pad 3: COL_08 -> COL_02
- A41 pad 4: COL_07 -> COL_03
- A41 pad 5: COL_06 -> ROW_0
- A41 pad 6: COL_03 -> ROW_1
- A41 pad 7: COL_05 -> COL_04
- A41 pad 8: COL_04 -> ROW_2
- A41 pad 9: COL_02 -> COL_06
Routing:
- net COL_11: track 149.7 -> 0.00 mm, vias 6 -> 0
- net GND: track 1150.6 -> 1258.3 mm, vias 9 -> 16
- net COL_10: track 122.5 -> 198.0 mm, vias 2 -> 3
- net COL_09: track 126.8 -> 190.2 mm, vias 4 -> 2
- net DIN: track 202.5 -> 141.2 mm, vias 2 -> 3
- net ROW_0: track 329.3 -> 268.7 mm, vias 2 -> 1
- net ROW_1: track 298.6 -> 238.4 mm, vias 2 -> 1
- net COL_07: track 49.9 -> 105.9 mm, vias 4 -> 2
- net Net-(A32-DOUT): track 31.4 -> 80.2 mm, vias 0 -> 4
- net COL_08: track 101.3 -> 149.8 mm, vias 6 -> 2
- net Net-(A33-DOUT): track 239.9 -> 288.1 mm
- net COL_04: track 90.4 -> 52.0 mm, vias 4 -> 0
- net COL_00: track 199.9 -> 168.2 mm, vias 4 -> 3
- net Net-(A23-DOUT): track 228.5 -> 258.5 mm
- net COL_01: track 173.7 -> 148.3 mm, vias 5 -> 3
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Other:
- board size 239.5 x 78 mm -> 239.5 x 187.5 mm
- board text added: "Just 40"
- board text added: "Mark I"
