File: kicad/just-40-mark03/just-40-mark03.kicad_pcb (KiCad board)
At the start: 2 copper layers, 230 x 181.2 mm, 125 parts

Commit message: wips
Parts:
- removed A10, A11, A12, A24, A25, A26, A27, A28, A29, A30, A31, A32, A33, A8, A9: KS-33-1U-LED-left, just-40-mark03:KS-33-1U-LED-left
- removed A13, A14, A15, A16, A17, A18, A19, A20, A21, A22, A23, A34, A35, A36, A37, A38, A39, A40: KS-33-1U-LED-right, just-40-mark03:KS-33-1U-LED-right
- removed A41: RP2350-Zero, just-40-mark03:RP2350-Tiny-SMD
- removed A42: SN74AHCT1G125DBVR, just-40-mark03:SN74AHCT1G125DBVR
- removed C1, C10, C11, C12, C13, C14, C15, C2, C3, C4, C5, C6, C7, C8, C9: ~, just-40-mark03:C410C104Z5U5TA7200
- removed H15, H16, H24, H25, H26, H27: mount-hole, just-40-mark03:hole-mount
- removed H17, H18, H19, H20, H21: mount-hole, just-40-mark03:hole-foot
- removed H22: RP2350-Tiny-USB, just-40-mark03:RP2350-Tiny-USB-2
- removed H23: RP2350-Tiny-USB-ref, just-40-mark03:RP2350-Tiny-USB-ref2
- added SW1: ~, just-40-mark03:KS-33-1U, F.Cu at (57.0, 38.0)
- added SW10: ~, just-40-mark03:KS-33-1U, F.Cu at (228.0, 38.0)
- added SW11: ~, just-40-mark03:KS-33-1U, F.Cu at (247.0, 38.0)
- added SW12: ~, just-40-mark03:KS-33-1U, F.Cu at (266.0, 38.0)
- added SW13: ~, just-40-mark03:KS-33-1U, F.Cu at (66.5, 57.0)
- added SW14: ~, just-40-mark03:KS-33-1U, F.Cu at (85.5, 57.0)
- added SW15: ~, just-40-mark03:KS-33-1U, F.Cu at (104.5, 57.0)
- added SW16: ~, just-40-mark03:KS-33-1U, F.Cu at (123.5, 57.0)
- added SW17: ~, just-40-mark03:KS-33-1U, F.Cu at (142.5, 57.0)
- added SW18: ~, just-40-mark03:KS-33-1U, F.Cu at (161.5, 57.0)
- added SW19: ~, just-40-mark03:KS-33-1U, F.Cu at (180.5, 57.0)
- added SW2: ~, just-40-mark03:KS-33-1U, F.Cu at (76.0, 38.0)
- added SW20: ~, just-40-mark03:KS-33-1U, F.Cu at (199.5, 57.0)
- added SW21: ~, just-40-mark03:KS-33-1U, F.Cu at (218.5, 57.0)
- added SW22: ~, just-40-mark03:KS-33-1U, F.Cu at (237.5, 57.0)
- added SW23: ~, just-40-mark03:KS-33-1U, F.Cu at (256.5, 57.0)
- added SW24: ~, just-40-mark03:KS-33-1U, F.Cu at (76.0, 76.0)
- added SW25: ~, just-40-mark03:KS-33-1U, F.Cu at (95.0, 76.0)
- added SW26: ~, just-40-mark03:KS-33-1U, F.Cu at (114.0, 76.0)
- added SW27: ~, just-40-mark03:KS-33-1U, F.Cu at (133.0, 76.0)
- added SW28: ~, just-40-mark03:KS-33-1U, F.Cu at (152.0, 76.0)
- added SW29: ~, just-40-mark03:KS-33-1U, F.Cu at (171.0, 76.0)
- added SW3: ~, just-40-mark03:KS-33-1U, F.Cu at (95.0, 38.0)
- added SW30: ~, just-40-mark03:KS-33-1U, F.Cu at (190.0, 76.0)
- added SW31: ~, just-40-mark03:KS-33-1U, F.Cu at (209.0, 76.0)
- added SW32: ~, just-40-mark03:KS-33-1U, F.Cu at (228.0, 76.0)
- added SW33: ~, just-40-mark03:KS-33-1U, F.Cu at (247.0, 76.0)
- added SW34: ~, just-40-mark03:KS-33-1U, F.Cu at (99.8, 95.0)
- added SW35: ~, just-40-mark03:KS-33-1U, F.Cu at (118.8, 95.0)
- added SW36: ~, just-40-mark03:KS-33-1U, F.Cu at (137.8, 95.0)
- added SW37: ~, just-40-mark03:KS-33-1U, F.Cu at (161.5, 95.0)
- added SW38: ~, just-40-mark03:KS-33-1U, F.Cu at (185.2, 95.0)
- added SW39: ~, just-40-mark03:KS-33-1U, F.Cu at (204.2, 95.0)
- added SW4: ~, just-40-mark03:KS-33-1U, F.Cu at (114.0, 38.0)
- added SW40: ~, just-40-mark03:KS-33-1U, F.Cu at (223.2, 95.0)
- added SW5: ~, just-40-mark03:KS-33-1U, F.Cu at (133.0, 38.0)
- added SW6: ~, just-40-mark03:KS-33-1U, F.Cu at (152.0, 38.0)
- added SW7: ~, just-40-mark03:KS-33-1U, F.Cu at (171.0, 38.0)
- added SW8: ~, just-40-mark03:KS-33-1U, F.Cu at (190.0, 38.0)
- added SW9: ~, just-40-mark03:KS-33-1U, F.Cu at (209.0, 38.0)
- A1: value KS-33-1U-LED-left -> RP2350-Zero; footprint just-40-mark03:KS-33-1U-LED-left -> just-40-mark03:RP2350-Tiny-SMD
- A2, A3, A4, A5, A6, A7: value KS-33-1U-LED-left -> neopixel; footprint just-40-mark03:KS-33-1U-LED-left -> just-40-mark03:SK6812MINI-E
- H10, H11, H12, H13, H9: footprint just-40-mark03:hole-mount -> just-40-mark03:hole-foot
- H14: value mount-hole -> RP2350-Tiny-USB; footprint just-40-mark03:hole-mount -> just-40-mark03:RP2350-Tiny-USB-4
- R1: value RR01JR33TB -> R; footprint just-40-mark03:RR01JR33TB -> just-40-mark03:330_ohm
- moved H14 235.6 mm to (161.5, 25.8), turned to -90 degrees
- moved A1 206.6 mm to (265.2, 80.8), turned to -90 degrees
- moved H13 205.5 mm to (161.5, 66.5)
- moved H10 200.7 mm to (256.5, 32.5)
- moved H11 159.0 mm to (66.5, 100.5)
- moved H9 152.8 mm to (66.5, 32.5)
- moved D18 142.2 mm to (56.0, 22.8)
- moved D36 141.6 mm to (81.0, 22.8)
- moved A2 140.7 mm to (218.5, 85.5)
- moved D29 138.1 mm to (262.0, 22.8)
- moved D37 128.2 mm to (182.0, 22.8)
- moved D39 127.5 mm to (217.0, 22.8)
- moved D38 127.4 mm to (197.0, 22.8)
- moved D34 127.4 mm to (111.0, 22.8)
- moved D35 127.3 mm to (126.0, 22.8)
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Connections:
- A1 pad 1: V_LED -> COL_04
- A1 pad 2: Net-(A1-DOUT) -> COL_05
- A1 pad 3: GND -> COL_06
- A1 pad 4: Net-(A1-DIN) -> COL_07
- A2 pad 1: V_LED -> 3V3
- A2 pad 2: Net-(A1-DIN) -> Net-(A2-DOUT)
- A3 pad 1: V_LED -> 3V3
- A3 pad 2: Net-(A2-DIN) -> Net-(A3-DOUT)
- A3 pad 4: Net-(A3-DIN) -> Net-(A2-DOUT)
- A4 pad 1: V_LED -> 3V3
- A4 pad 2: Net-(A3-DIN) -> Net-(A4-DOUT)
- A4 pad 4: Net-(A4-DIN) -> Net-(A3-DOUT)
- A5 pad 1: V_LED -> 3V3
- A5 pad 2: Net-(A4-DIN) -> Net-(A5-DOUT)
- A5 pad 4: Net-(A5-DIN) -> Net-(A4-DOUT)
- A6 pad 1: V_LED -> 3V3
- A6 pad 2: Net-(A5-DIN) -> Net-(A6-DOUT)
- A6 pad 4: Net-(A6-DIN) -> Net-(A5-DOUT)
- A7 pad 1: V_LED -> 3V3
- A7 pad 2: Net-(A6-DIN) -> unconnected-(A7-DOUT-Pad2)_1
- A7 pad 4: Net-(A7-DIN) -> Net-(A6-DOUT)
- D1 pad A: Net-(A1-PadB) -> Net-(SW1-B)
- D2 pad A: Net-(A2-PadB) -> Net-(SW2-B)
- D3 pad A: Net-(A3-PadB) -> Net-(SW3-B)
- D4 pad A: Net-(A4-PadB) -> Net-(SW4-B)
- D5 pad A: Net-(A5-PadB) -> Net-(SW5-B)
- D6 pad A: Net-(A6-PadB) -> Net-(SW6-B)
- D7 pad A: Net-(A7-PadB) -> Net-(SW7-B)
- R1 pad 2: Net-(A42-Y) -> Net-(A2-DIN)
Routing:
- net Net-(A5-DOUT): track 0.00 -> 184.8 mm
- net ROW_2: track 219.6 -> 389.5 mm, vias 10 -> 14
- net Net-(SW29-B): track 6.37 -> 173.4 mm, vias 0 -> 7
- net DIN: track 11.2 -> 169.4 mm, vias 0 -> 3
- net Net-(SW18-B): track 6.37 -> 163.9 mm, vias 0 -> 5
- net Net-(SW36-B): track 6.37 -> 156.4 mm, vias 0 -> 4
- net ROW_3: track 182.1 -> 323.9 mm, vias 7 -> 11
- net Net-(A2-DIN): track 13.8 -> 152.2 mm, vias 0 -> 5
- net Net-(SW17-B): track 6.37 -> 116.4 mm, vias 0 -> 5
- net Net-(A2-DOUT): track 0.00 -> 108.5 mm
- net Net-(SW39-B): track 6.37 -> 107.7 mm, vias 0 -> 7
- net Net-(SW38-B): track 6.37 -> 106.7 mm, vias 0 -> 7
- net Net-(SW40-B): track 6.37 -> 104.7 mm, vias 0 -> 9
- net Net-(SW31-B): track 6.37 -> 104.4 mm, vias 0 -> 7
- net Net-(SW34-B): track 6.37 -> 97.2 mm, vias 0 -> 7
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- added copper zone on F.Cu, net 3V3
- removed copper zone on F.Cu, net V_LED
Other:
- board size 230 x 181.2 mm -> 230 x 89 mm
