File: kicad/just-40-mark03/just-40-mark03.kicad_pcb (KiCad board)
At the start: 2 copper layers, 230 x 101.5 mm, 101 parts

Commit message: wips
Parts:
- removed A27: RP2350-Zero, just-40-mark03:RP2350-Zero_1
- added A1: RP2350-Zero, just-40-mark03:RP2350-Zero_5, F.Cu at (161.5, 36.0)
- added A2: RP2350-Zero, just-40-mark03:RP2350-Tiny-SMD_1, F.Cu at (251.8, 209.5)
- added A3: RP2350-Zero, just-40-mark03:RP2350-Tiny-THT_2, F.Cu at (241.2, 250.0)
- added A4: RP2350-Zero, just-40-mark03:RP2350-Tiny-SMD_1, F.Cu at (263.5, 549.0)
- added D100: 1N4148, just-40-mark03:1N4148_2, F.Cu at (186.5, 246.5)
- added D101: 1N4148, just-40-mark03:1N4148_2, F.Cu at (202.8, 246.5)
- added D102: 1N4148, just-40-mark03:1N4148_2, F.Cu at (209.2, 246.5)
- added D103: 1N4148, just-40-mark03:1N4148_2, F.Cu at (222.2, 246.5)
- added D104: 1N4148, just-40-mark03:1N4148_2, F.Cu at (78.0, 246.5)
- added D105: 1N4148, just-40-mark03:1N4148_2, F.Cu at (87.8, 246.5)
- added D106: 1N4148, just-40-mark03:1N4148_2, F.Cu at (100.8, 246.5)
- added D107: 1N4148, just-40-mark03:1N4148_2, F.Cu at (113.8, 246.5)
- added D108: 1N4148, just-40-mark03:1N4148_2, F.Cu at (130.0, 246.5)
- added D109: 1N4148, just-40-mark03:1N4148_2, F.Cu at (143.0, 246.5)
- added D110: 1N4148, just-40-mark03:1N4148_2, F.Cu at (176.8, 246.5)
- added D111: 1N4148, just-40-mark03:1N4148_2, F.Cu at (189.8, 246.5)
- added D112: 1N4148, just-40-mark03:1N4148_2, F.Cu at (206.0, 246.5)
- added D113: 1N4148, just-40-mark03:1N4148_2, F.Cu at (225.5, 246.5)
- added D114: 1N4148, just-40-mark03:1N4148_2, F.Cu at (91.0, 246.5)
- added D115: 1N4148, just-40-mark03:1N4148_2, F.Cu at (104.0, 246.5)
- added D116: 1N4148, just-40-mark03:1N4148_2, F.Cu at (117.0, 246.5)
- added D117: 1N4148, just-40-mark03:1N4148_2, F.Cu at (133.2, 246.5)
- added D118: 1N4148, just-40-mark03:1N4148_2, F.Cu at (146.2, 246.5)
- added D119: 1N4148, just-40-mark03:1N4148_2, F.Cu at (180.0, 246.5)
- added D120: 1N4148, just-40-mark03:1N4148_2, F.Cu at (193.0, 246.5)
- added D121: 1N4148, just-40-mark03:1N4148_2, F.Cu at (65.2, 500.0)
- added D122: 1N4148, just-40-mark03:1N4148_2, F.Cu at (84.2, 500.0)
- added D123: 1N4148, just-40-mark03:1N4148_2, F.Cu at (103.2, 500.0)
- added D124: 1N4148, just-40-mark03:1N4148_2, F.Cu at (122.2, 500.0)
- added D125: 1N4148, just-40-mark03:1N4148_2, F.Cu at (141.2, 500.0)
- added D126: 1N4148, just-40-mark03:1N4148_2, F.Cu at (143.8, 500.0)
- added D127: 1N4148, just-40-mark03:1N4148_2, F.Cu at (179.2, 500.0)
- added D128: 1N4148, just-40-mark03:1N4148_2, F.Cu at (198.2, 500.0)
- added D129: 1N4148, just-40-mark03:1N4148_2, F.Cu at (217.2, 500.0)
- added D130: 1N4148, just-40-mark03:1N4148_2, F.Cu at (236.2, 500.0)
- added D131: 1N4148, just-40-mark03:1N4148_2, F.Cu at (255.2, 500.0)
- added D132: 1N4148, just-40-mark03:1N4148_2, F.Cu at (274.2, 500.0)
- added D133: 1N4148, just-40-mark03:1N4148_2, F.Cu at (74.8, 519.0)
- added D134: 1N4148, just-40-mark03:1N4148_2, F.Cu at (93.8, 519.0)
- added D135: 1N4148, just-40-mark03:1N4148_2, F.Cu at (112.8, 519.0)
- added D136: 1N4148, just-40-mark03:1N4148_2, F.Cu at (131.8, 519.0)
- added D137: 1N4148, just-40-mark03:1N4148_2, F.Cu at (150.8, 519.0)
- added D138: 1N4148, just-40-mark03:1N4148_2, F.Cu at (169.8, 519.0)
- added D139: 1N4148, just-40-mark03:1N4148_2, F.Cu at (188.8, 519.0)
- added D140: 1N4148, just-40-mark03:1N4148_2, F.Cu at (207.8, 519.0)
- added D141: 1N4148, just-40-mark03:1N4148_2, F.Cu at (226.8, 519.0)
- added D142: 1N4148, just-40-mark03:1N4148_2, F.Cu at (245.8, 519.0)
- added D143: 1N4148, just-40-mark03:1N4148_2, F.Cu at (264.8, 519.0)
- added D144: 1N4148, just-40-mark03:1N4148_2, F.Cu at (84.2, 538.0)
- added D145: 1N4148, just-40-mark03:1N4148_2, F.Cu at (103.2, 538.0)
- added D146: 1N4148, just-40-mark03:1N4148_2, F.Cu at (122.2, 538.0)
- added D147: 1N4148, just-40-mark03:1N4148_2, F.Cu at (141.2, 538.0)
- added D148: 1N4148, just-40-mark03:1N4148_2, F.Cu at (160.2, 538.0)
- added D149: 1N4148, just-40-mark03:1N4148_2, F.Cu at (179.2, 538.0)
- added D150: 1N4148, just-40-mark03:1N4148_2, F.Cu at (198.2, 538.0)
- added D151: 1N4148, just-40-mark03:1N4148_2, F.Cu at (217.2, 538.0)
- added D152: 1N4148, just-40-mark03:1N4148_2, F.Cu at (236.2, 538.0)
- added D153: 1N4148, just-40-mark03:1N4148_2, F.Cu at (238.8, 538.0)
- added D154: 1N4148, just-40-mark03:1N4148_2, F.Cu at (112.8, 557.0)
- added D155: 1N4148, just-40-mark03:1N4148_2, F.Cu at (131.8, 557.0)
- added D156: 1N4148, just-40-mark03:1N4148_2, F.Cu at (150.8, 557.0)
- added D157: 1N4148, just-40-mark03:1N4148_2, F.Cu at (169.8, 557.0)
- added D158: 1N4148, just-40-mark03:1N4148_2, F.Cu at (188.8, 557.0)
- added D159: 1N4148, just-40-mark03:1N4148_2, F.Cu at (207.8, 557.0)
- added D160: 1N4148, just-40-mark03:1N4148_2, F.Cu at (226.8, 557.0)
- added D41: 1N4148, just-40-mark03:1N4148_2, F.Cu at (65.2, 153.0)
- added D42: 1N4148, just-40-mark03:1N4148_2, F.Cu at (84.2, 153.0)
- added D43: 1N4148, just-40-mark03:1N4148_2, F.Cu at (103.2, 153.0)
- added D44: 1N4148, just-40-mark03:1N4148_2, F.Cu at (105.8, 153.0)
- added D45: 1N4148, just-40-mark03:1N4148_2, F.Cu at (141.2, 153.0)
- added D46: 1N4148, just-40-mark03:1N4148_2, F.Cu at (143.8, 153.0)
- added D47: 1N4148, just-40-mark03:1N4148_2, F.Cu at (179.2, 153.0)
- added D48: 1N4148, just-40-mark03:1N4148_2, F.Cu at (181.8, 153.0)
- added D49: 1N4148, just-40-mark03:1N4148_2, F.Cu at (217.2, 153.0)
- added D50: 1N4148, just-40-mark03:1N4148_2, F.Cu at (236.2, 153.0)
- added D51: 1N4148, just-40-mark03:1N4148_2, F.Cu at (255.2, 153.0)
- added D52: 1N4148, just-40-mark03:1N4148_2, F.Cu at (257.8, 153.0)
- added D53: 1N4148, just-40-mark03:1N4148_2, F.Cu at (74.8, 172.0)
- added D54: 1N4148, just-40-mark03:1N4148_2, F.Cu at (93.8, 172.0)
- added D55: 1N4148, just-40-mark03:1N4148_2, F.Cu at (112.8, 172.0)
- added D56: 1N4148, just-40-mark03:1N4148_2, F.Cu at (131.8, 172.0)
- added D57: 1N4148, just-40-mark03:1N4148_2, F.Cu at (150.8, 172.0)
- added D58: 1N4148, just-40-mark03:1N4148_2, F.Cu at (169.8, 172.0)
- added D59: 1N4148, just-40-mark03:1N4148_2, F.Cu at (188.8, 172.0)
- added D60: 1N4148, just-40-mark03:1N4148_2, F.Cu at (207.8, 172.0)
- added D61: 1N4148, just-40-mark03:1N4148_2, F.Cu at (226.8, 172.0)
- added D62: 1N4148, just-40-mark03:1N4148_2, F.Cu at (245.8, 172.0)
- added D63: 1N4148, just-40-mark03:1N4148_2, F.Cu at (264.8, 172.0)
- added D64: 1N4148, just-40-mark03:1N4148_2, F.Cu at (84.2, 191.0)
- added D65: 1N4148, just-40-mark03:1N4148_2, F.Cu at (103.2, 191.0)
- added D66: 1N4148, just-40-mark03:1N4148_2, F.Cu at (122.2, 191.0)
- added D67: 1N4148, just-40-mark03:1N4148_2, F.Cu at (141.2, 191.0)
- added D68: 1N4148, just-40-mark03:1N4148_2, F.Cu at (160.2, 191.0)
- added D69: 1N4148, just-40-mark03:1N4148_2, F.Cu at (179.2, 191.0)
- added D70: 1N4148, just-40-mark03:1N4148_2, F.Cu at (198.2, 191.0)
- added D71: 1N4148, just-40-mark03:1N4148_2, F.Cu at (217.2, 191.0)
- added D72: 1N4148, just-40-mark03:1N4148_2, F.Cu at (236.2, 191.0)
- added D73: 1N4148, just-40-mark03:1N4148_2, F.Cu at (255.2, 191.0)
- added D74: 1N4148, just-40-mark03:1N4148_2, F.Cu at (112.8, 210.0)
- added D75: 1N4148, just-40-mark03:1N4148_2, F.Cu at (115.2, 210.0)
- added D76: 1N4148, just-40-mark03:1N4148_2, F.Cu at (150.8, 210.0)
- added D77: 1N4148, just-40-mark03:1N4148_2, F.Cu at (169.8, 210.0)
- added D78: 1N4148, just-40-mark03:1N4148_2, F.Cu at (172.2, 210.0)
- added D79: 1N4148, just-40-mark03:1N4148_2, F.Cu at (207.8, 210.0)
- added D80: 1N4148, just-40-mark03:1N4148_2, F.Cu at (226.8, 210.0)
- added D81: 1N4148, just-40-mark03:1N4148_2, F.Cu at (71.5, 246.5)
- added D82: 1N4148, just-40-mark03:1N4148_2, F.Cu at (81.2, 246.5)
- added D83: 1N4148, just-40-mark03:1N4148_2, F.Cu at (94.2, 246.5)
- added D84: 1N4148, just-40-mark03:1N4148_2, F.Cu at (107.2, 246.5)
- added D85: 1N4148, just-40-mark03:1N4148_2, F.Cu at (120.2, 246.5)
- added D86: 1N4148, just-40-mark03:1N4148_2, F.Cu at (136.5, 246.5)
- added D87: 1N4148, just-40-mark03:1N4148_2, F.Cu at (149.5, 246.5)
- added D88: 1N4148, just-40-mark03:1N4148_2, F.Cu at (183.2, 246.5)
- added D89: 1N4148, just-40-mark03:1N4148_2, F.Cu at (196.2, 246.5)
- added D90: 1N4148, just-40-mark03:1N4148_2, F.Cu at (215.8, 246.5)
- added D91: 1N4148, just-40-mark03:1N4148_2, F.Cu at (212.5, 246.5)
- added D92: 1N4148, just-40-mark03:1N4148_2, F.Cu at (219.0, 246.5)
- added D93: 1N4148, just-40-mark03:1N4148_2, F.Cu at (74.8, 246.5)
- added D94: 1N4148, just-40-mark03:1N4148_2, F.Cu at (84.5, 246.5)
- added D95: 1N4148, just-40-mark03:1N4148_2, F.Cu at (97.5, 246.5)
- added D96: 1N4148, just-40-mark03:1N4148_2, F.Cu at (110.5, 246.5)
- added D97: 1N4148, just-40-mark03:1N4148_2, F.Cu at (126.8, 246.5)
- added D98: 1N4148, just-40-mark03:1N4148_2, F.Cu at (139.8, 246.5)
- added D99: 1N4148, just-40-mark03:1N4148_2, F.Cu at (173.5, 246.5)
- added G***: LOGO, just-40-mark03:penguin-sword-40, F.Cu at (161.5, 628.5)
- added G***: LOGO, just-40-mark03:penguin-sword-40, F.Cu at (57.0, 200.5)
- added H10: mount-hole, just-40-mark03:hole-foot, F.Cu at (266.0, 37.0)
- added H11: mount-hole, just-40-mark03:hole-foot, F.Cu at (57.0, 112.0)
- added H12: mount-hole, just-40-mark03:hole-foot, F.Cu at (133.0, 112.0)
- added H13: mount-hole, just-40-mark03:hole-foot, F.Cu at (133.0, 37.0)
- added H14: mount-hole, just-40-mark03:hole-foot, F.Cu at (266.0, 112.0)
- added H15: mount-hole, just-40-mark03:hole-foot, F.Cu at (190.0, 37.0)
- added H16: mount-hole, just-40-mark03:hole-foot, F.Cu at (190.0, 112.0)
- added H17: mount-hole, just-40-mark03:hole-mount, F.Cu at (49.5, 144.0)
- added H18: mount-hole, just-40-mark03:hole-mount, F.Cu at (199.5, 144.0)
- added H19: mount-hole, just-40-mark03:hole-mount, F.Cu at (49.5, 217.5)
- added H20: mount-hole, just-40-mark03:hole-mount, F.Cu at (190.0, 217.5)
- added H21: mount-hole, just-40-mark03:hole-mount, F.Cu at (123.5, 144.0)
- added H22: mount-hole, just-40-mark03:hole-mount, F.Cu at (273.5, 144.0)
- added H23: mount-hole, just-40-mark03:hole-mount, F.Cu at (133.0, 217.5)
- added H24: mount-hole, just-40-mark03:hole-mount, F.Cu at (273.5, 217.5)
- added H25: mount-hole, just-40-mark03:hole-foot, F.Cu at (54.0, 148.5)
- added H26: mount-hole, just-40-mark03:hole-foot, F.Cu at (190.0, 211.0)
- added H27: mount-hole, just-40-mark03:hole-foot, F.Cu at (199.5, 150.5)
- added H28: mount-hole, just-40-mark03:hole-foot, F.Cu at (54.0, 213.0)
- added H29: mount-hole, just-40-mark03:hole-foot, F.Cu at (123.5, 150.5)
- added H30: mount-hole, just-40-mark03:hole-foot, F.Cu at (269.0, 213.0)
- added H31: mount-hole, just-40-mark03:hole-foot, F.Cu at (269.0, 148.5)
- added H32: mount-hole, just-40-mark03:hole-foot, F.Cu at (133.0, 211.0)
- added H33: RP2350-Tiny-USB, just-40-mark03:RP2350-Tiny-USB-3, F.Cu at (161.5, 150.5)
- added H34: mount-hole, just-40-mark03:hole-mount, F.Cu at (181.1, 376.6)
- added H35: mount-hole, just-40-mark03:hole-mount, F.Cu at (181.1, 381.6)
- added H36: mount-hole, just-40-mark03:hole-mount, F.Cu at (186.2, 376.6)
- added H37: mount-hole, just-40-mark03:hole-mount, F.Cu at (186.2, 381.6)
- added H38: mount-hole, just-40-mark03:hole-mount, F.Cu at (191.2, 376.6)
- added H39: mount-hole, just-40-mark03:hole-mount, F.Cu at (191.2, 381.6)
- added H40: mount-hole, just-40-mark03:hole-mount, F.Cu at (196.3, 376.6)
- added H41: mount-hole, just-40-mark03:hole-mount, F.Cu at (196.3, 381.6)
- added H42: mount-hole, just-40-mark03:hole-mount, F.Cu at (48.5, 253.5)
- added H43: mount-hole, just-40-mark03:hole-mount, F.Cu at (123.5, 253.5)
- added H44: mount-hole, just-40-mark03:hole-mount, F.Cu at (199.5, 253.5)
- added H45: mount-hole, just-40-mark03:hole-mount, F.Cu at (274.5, 253.5)
- added H46: mount-hole, just-40-mark03:hole-mount, F.Cu at (48.5, 327.0)
- added H47: mount-hole, just-40-mark03:hole-mount, F.Cu at (133.0, 327.0)
- added H48: mount-hole, just-40-mark03:hole-mount, F.Cu at (190.0, 327.0)
- added H49: mount-hole, just-40-mark03:hole-mount, F.Cu at (274.5, 327.0)
- added H50: mount-hole, just-40-mark03:hole-foot, F.Cu at (145.3, 368.3)
- added H51: mount-hole, just-40-mark03:hole-foot, F.Cu at (145.3, 377.4)
- added H52: mount-hole, just-40-mark03:hole-foot, F.Cu at (145.3, 386.5)
- added H53: mount-hole, just-40-mark03:hole-foot, F.Cu at (145.3, 395.6)
- added H54: mount-hole, just-40-mark03:hole-foot, F.Cu at (145.3, 404.7)
- added H55: mount-hole, just-40-mark03:hole-foot, F.Cu at (154.4, 368.3)
- added H56: mount-hole, just-40-mark03:hole-foot, F.Cu at (154.4, 377.4)
- added H57: mount-hole, just-40-mark03:hole-foot, F.Cu at (154.4, 386.5)
- added H58: mount-hole, just-40-mark03:hole-foot, F.Cu at (154.4, 395.6)
- added H59: mount-hole, just-40-mark03:hole-foot, F.Cu at (154.4, 404.7)
- added H60: RP2350-Tiny-USB, just-40-mark03:RP2350-Tiny-USB, F.Cu at (161.5, 249.5)
- added H61: mount-hole, just-40-mark03:hole-mount, F.Cu at (48.5, 491.5)
- added H62: mount-hole, just-40-mark03:hole-mount, F.Cu at (123.5, 491.5)
- added H63: mount-hole, just-40-mark03:hole-mount, F.Cu at (199.5, 491.5)
- added H64: mount-hole, just-40-mark03:hole-mount, F.Cu at (274.5, 491.5)
- added H76: mount-hole, just-40-mark03:hole-foot, F.Cu at (270.0, 661.0)
- added H77: mount-hole, just-40-mark03:hole-mount, F.Cu at (48.5, 591.5)
- added H78: mount-hole, just-40-mark03:hole-mount, F.Cu at (123.5, 591.5)
- added H79: mount-hole, just-40-mark03:hole-mount, F.Cu at (199.5, 591.5)
- added H80: mount-hole, just-40-mark03:hole-mount, F.Cu at (274.5, 591.5)
- added H81: mount-hole, just-40-mark03:hole-mount, F.Cu at (48.5, 665.5)
- added H82: mount-hole, just-40-mark03:hole-mount, F.Cu at (133.0, 665.5)
- added H83: mount-hole, just-40-mark03:hole-mount, F.Cu at (190.0, 665.5)
- added H84: mount-hole, just-40-mark03:hole-mount, F.Cu at (274.5, 665.5)
- added H85: RP2350-Tiny-USB, just-40-mark03:RP2350-Tiny-USB-ref_4, F.Cu at (161.5, 497.5)
- added H86: RP2350-Tiny-USB, just-40-mark03:RP2350-Tiny-USB, F.Cu at (161.5, 597.5)
- added H9: mount-hole, just-40-mark03:hole-foot, F.Cu at (57.0, 37.0)
- added SW100: ~, just-40-mark03:KS-33-1U_4, F.Cu at (199.5, 281.0)
- added SW101: ~, just-40-mark03:KS-33-1U_4, F.Cu at (218.5, 281.0)
- added SW102: ~, just-40-mark03:KS-33-1U_4, F.Cu at (237.5, 281.0)
- added SW103: ~, just-40-mark03:KS-33-1U_4, F.Cu at (256.5, 281.0)
- added SW104: ~, just-40-mark03:KS-33-1U_4, F.Cu at (76.0, 300.0)
- added SW105: ~, just-40-mark03:KS-33-1U_4, F.Cu at (95.0, 300.0)
- added SW106: ~, just-40-mark03:KS-33-1U_4, F.Cu at (114.0, 300.0)
- added SW107: ~, just-40-mark03:KS-33-1U_4, F.Cu at (133.0, 300.0)
- added SW108: ~, just-40-mark03:KS-33-1U_4, F.Cu at (152.0, 300.0)
- added SW109: ~, just-40-mark03:KS-33-1U_4, F.Cu at (171.0, 300.0)
- added SW110: ~, just-40-mark03:KS-33-1U_4, F.Cu at (190.0, 300.0)
- added SW111: ~, just-40-mark03:KS-33-1U_4, F.Cu at (209.0, 300.0)
- added SW112: ~, just-40-mark03:KS-33-1U_4, F.Cu at (228.0, 300.0)
- added SW113: ~, just-40-mark03:KS-33-1U_4, F.Cu at (247.0, 300.0)
- added SW114: ~, just-40-mark03:KS-33-1U_4, F.Cu at (104.5, 319.0)
- added SW115: ~, just-40-mark03:KS-33-1U_4, F.Cu at (123.5, 319.0)
- added SW116: ~, just-40-mark03:KS-33-1U_4, F.Cu at (142.5, 319.0)
- added SW117: ~, just-40-mark03:KS-33-1U_4, F.Cu at (161.5, 319.0)
- added SW118: ~, just-40-mark03:KS-33-1U_4, F.Cu at (180.5, 319.0)
- added SW119: ~, just-40-mark03:KS-33-1U_4, F.Cu at (199.5, 319.0)
- added SW120: ~, just-40-mark03:KS-33-1U_4, F.Cu at (218.5, 319.0)
- added SW121: ~, just-40-mark03:KS-33-1U_4, F.Cu at (57.0, 500.0)
- added SW122: ~, just-40-mark03:KS-33-1U_4, F.Cu at (76.0, 500.0)
- added SW123: ~, just-40-mark03:KS-33-1U_4, F.Cu at (95.0, 500.0)
- added SW124: ~, just-40-mark03:KS-33-1U_4, F.Cu at (114.0, 500.0)
- added SW125: ~, just-40-mark03:KS-33-1U_4, F.Cu at (133.0, 500.0)
- added SW126: ~, just-40-mark03:KS-33-1U_4, F.Cu at (152.0, 500.0)
- added SW127: ~, just-40-mark03:KS-33-1U_4, F.Cu at (171.0, 500.0)
- added SW128: ~, just-40-mark03:KS-33-1U_4, F.Cu at (190.0, 500.0)
- added SW129: ~, just-40-mark03:KS-33-1U_4, F.Cu at (209.0, 500.0)
- added SW130: ~, just-40-mark03:KS-33-1U_4, F.Cu at (228.0, 500.0)
- added SW131: ~, just-40-mark03:KS-33-1U_4, F.Cu at (247.0, 500.0)
- added SW132: ~, just-40-mark03:KS-33-1U_4, F.Cu at (266.0, 500.0)
- added SW133: ~, just-40-mark03:KS-33-1U_4, F.Cu at (66.5, 519.0)
- added SW134: ~, just-40-mark03:KS-33-1U_4, F.Cu at (85.5, 519.0)
- added SW135: ~, just-40-mark03:KS-33-1U_4, F.Cu at (104.5, 519.0)
- added SW136: ~, just-40-mark03:KS-33-1U_4, F.Cu at (123.5, 519.0)
- added SW137: ~, just-40-mark03:KS-33-1U_4, F.Cu at (142.5, 519.0)
- added SW138: ~, just-40-mark03:KS-33-1U_4, F.Cu at (161.5, 519.0)
- added SW139: ~, just-40-mark03:KS-33-1U_4, F.Cu at (180.5, 519.0)
- added SW140: ~, just-40-mark03:KS-33-1U_4, F.Cu at (199.5, 519.0)
- added SW141: ~, just-40-mark03:KS-33-1U_4, F.Cu at (218.5, 519.0)
- added SW142: ~, just-40-mark03:KS-33-1U_4, F.Cu at (237.5, 519.0)
- added SW143: ~, just-40-mark03:KS-33-1U_4, F.Cu at (256.5, 519.0)
- added SW144: ~, just-40-mark03:KS-33-1U_4, F.Cu at (76.0, 538.0)
- added SW145: ~, just-40-mark03:KS-33-1U_4, F.Cu at (95.0, 538.0)
- added SW146: ~, just-40-mark03:KS-33-1U_4, F.Cu at (114.0, 538.0)
- added SW147: ~, just-40-mark03:KS-33-1U_4, F.Cu at (133.0, 538.0)
- added SW148: ~, just-40-mark03:KS-33-1U_4, F.Cu at (152.0, 538.0)
- added SW149: ~, just-40-mark03:KS-33-1U_4, F.Cu at (171.0, 538.0)
- added SW150: ~, just-40-mark03:KS-33-1U_4, F.Cu at (190.0, 538.0)
- added SW151: ~, just-40-mark03:KS-33-1U_4, F.Cu at (209.0, 538.0)
- added SW152: ~, just-40-mark03:KS-33-1U_4, F.Cu at (228.0, 538.0)
- added SW153: ~, just-40-mark03:KS-33-1U_4, F.Cu at (247.0, 538.0)
- added SW154: ~, just-40-mark03:KS-33-1U_4, F.Cu at (104.5, 557.0)
- added SW155: ~, just-40-mark03:KS-33-1U_4, F.Cu at (123.5, 557.0)
- added SW156: ~, just-40-mark03:KS-33-1U_4, F.Cu at (142.5, 557.0)
- added SW157: ~, just-40-mark03:KS-33-1U_4, F.Cu at (161.5, 557.0)
- added SW158: ~, just-40-mark03:KS-33-1U_4, F.Cu at (180.5, 557.0)
- added SW159: ~, just-40-mark03:KS-33-1U_4, F.Cu at (199.5, 557.0)
- added SW160: ~, just-40-mark03:KS-33-1U_4, F.Cu at (218.5, 557.0)
- added SW41: ~, just-40-mark03:KS-33-1U_2, F.Cu at (57.0, 153.0)
- added SW42: ~, just-40-mark03:KS-33-1U_2, F.Cu at (76.0, 153.0)
- added SW43: ~, just-40-mark03:KS-33-1U_2, F.Cu at (95.0, 153.0)
- added SW44: ~, just-40-mark03:KS-33-1U_2, F.Cu at (114.0, 153.0)
- added SW45: ~, just-40-mark03:KS-33-1U_2, F.Cu at (133.0, 153.0)
- added SW46: ~, just-40-mark03:KS-33-1U_2, F.Cu at (152.0, 153.0)
- added SW47: ~, just-40-mark03:KS-33-1U_2, F.Cu at (171.0, 153.0)
- added SW48: ~, just-40-mark03:KS-33-1U_2, F.Cu at (190.0, 153.0)
- added SW49: ~, just-40-mark03:KS-33-1U_2, F.Cu at (209.0, 153.0)
- added SW50: ~, just-40-mark03:KS-33-1U_2, F.Cu at (228.0, 153.0)
- added SW51: ~, just-40-mark03:KS-33-1U_2, F.Cu at (247.0, 153.0)
- added SW52: ~, just-40-mark03:KS-33-1U_2, F.Cu at (266.0, 153.0)
- added SW53: ~, just-40-mark03:KS-33-1U_2, F.Cu at (66.5, 172.0)
- added SW54: ~, just-40-mark03:KS-33-1U_2, F.Cu at (85.5, 172.0)
- added SW55: ~, just-40-mark03:KS-33-1U_2, F.Cu at (104.5, 172.0)
- added SW56: ~, just-40-mark03:KS-33-1U_2, F.Cu at (123.5, 172.0)
- added SW57: ~, just-40-mark03:KS-33-1U_2, F.Cu at (142.5, 172.0)
- added SW58: ~, just-40-mark03:KS-33-1U_2, F.Cu at (161.5, 172.0)
- added SW59: ~, just-40-mark03:KS-33-1U_2, F.Cu at (180.5, 172.0)
- added SW60: ~, just-40-mark03:KS-33-1U_2, F.Cu at (199.5, 172.0)
- added SW61: ~, just-40-mark03:KS-33-1U_2, F.Cu at (218.5, 172.0)
- added SW62: ~, just-40-mark03:KS-33-1U_2, F.Cu at (237.5, 172.0)
- added SW63: ~, just-40-mark03:KS-33-1U_2, F.Cu at (256.5, 172.0)
- added SW64: ~, just-40-mark03:KS-33-1U_2, F.Cu at (76.0, 191.0)
- added SW65: ~, just-40-mark03:KS-33-1U_2, F.Cu at (95.0, 191.0)
- added SW66: ~, just-40-mark03:KS-33-1U_2, F.Cu at (114.0, 191.0)
- added SW67: ~, just-40-mark03:KS-33-1U_2, F.Cu at (133.0, 191.0)
- added SW68: ~, just-40-mark03:KS-33-1U_2, F.Cu at (152.0, 191.0)
- added SW69: ~, just-40-mark03:KS-33-1U_2, F.Cu at (171.0, 191.0)
- added SW70: ~, just-40-mark03:KS-33-1U_2, F.Cu at (190.0, 191.0)
- added SW71: ~, just-40-mark03:KS-33-1U_2, F.Cu at (209.0, 191.0)
- added SW72: ~, just-40-mark03:KS-33-1U_2, F.Cu at (228.0, 191.0)
- added SW73: ~, just-40-mark03:KS-33-1U_2, F.Cu at (247.0, 191.0)
- added SW74: ~, just-40-mark03:KS-33-1U_2, F.Cu at (104.5, 210.0)
- added SW75: ~, just-40-mark03:KS-33-1U_2, F.Cu at (123.5, 210.0)
- added SW76: ~, just-40-mark03:KS-33-1U_2, F.Cu at (142.5, 210.0)
- added SW77: ~, just-40-mark03:KS-33-1U_2, F.Cu at (161.5, 210.0)
- added SW78: ~, just-40-mark03:KS-33-1U_2, F.Cu at (180.5, 210.0)
- added SW79: ~, just-40-mark03:KS-33-1U_2, F.Cu at (199.5, 210.0)
- added SW80: ~, just-40-mark03:KS-33-1U_2, F.Cu at (218.5, 210.0)
- added SW81: ~, just-40-mark03:KS-33-1U_4, F.Cu at (57.0, 262.0)
- added SW82: ~, just-40-mark03:KS-33-1U_4, F.Cu at (76.0, 262.0)
- added SW83: ~, just-40-mark03:KS-33-1U_4, F.Cu at (95.0, 262.0)
- added SW84: ~, just-40-mark03:KS-33-1U_4, F.Cu at (114.0, 262.0)
- added SW85: ~, just-40-mark03:KS-33-1U_4, F.Cu at (133.0, 262.0)
- added SW86: ~, just-40-mark03:KS-33-1U_4, F.Cu at (152.0, 262.0)
- added SW87: ~, just-40-mark03:KS-33-1U_4, F.Cu at (171.0, 262.0)
- added SW88: ~, just-40-mark03:KS-33-1U_4, F.Cu at (190.0, 262.0)
- added SW89: ~, just-40-mark03:KS-33-1U_4, F.Cu at (209.0, 262.0)
- added SW90: ~, just-40-mark03:KS-33-1U_4, F.Cu at (228.0, 262.0)
- added SW91: ~, just-40-mark03:KS-33-1U_4, F.Cu at (247.0, 262.0)
- added SW92: ~, just-40-mark03:KS-33-1U_4, F.Cu at (266.0, 262.0)
- added SW93: ~, just-40-mark03:KS-33-1U_4, F.Cu at (66.5, 281.0)
- added SW94: ~, just-40-mark03:KS-33-1U_4, F.Cu at (85.5, 281.0)
- added SW95: ~, just-40-mark03:KS-33-1U_4, F.Cu at (104.5, 281.0)
- added SW96: ~, just-40-mark03:KS-33-1U_4, F.Cu at (123.5, 281.0)
- added SW97: ~, just-40-mark03:KS-33-1U_4, F.Cu at (142.5, 281.0)
- added SW98: ~, just-40-mark03:KS-33-1U_4, F.Cu at (161.5, 281.0)
- added SW99: ~, just-40-mark03:KS-33-1U_4, F.Cu at (180.5, 281.0)
- D1: renamed from D181; footprint just-40-mark03:1N4148 -> just-40-mark03:1N4148_2
- D10: renamed from D190; footprint just-40-mark03:1N4148 -> just-40-mark03:1N4148_2
- D11: renamed from D191; footprint just-40-mark03:1N4148 -> just-40-mark03:1N4148_2
- D12: renamed from D192; footprint just-40-mark03:1N4148 -> just-40-mark03:1N4148_2
- D13: renamed from D193; footprint just-40-mark03:1N4148 -> just-40-mark03:1N4148_2
- D14: renamed from D194; footprint just-40-mark03:1N4148 -> just-40-mark03:1N4148_2
- D15: renamed from D195; footprint just-40-mark03:1N4148 -> just-40-mark03:1N4148_2
- D16: renamed from D196; footprint just-40-mark03:1N4148 -> just-40-mark03:1N4148_2
- D17: renamed from D197; footprint just-40-mark03:1N4148 -> just-40-mark03:1N4148_2
- D18: renamed from D198; footprint just-40-mark03:1N4148 -> just-40-mark03:1N4148_2
- D19: renamed from D199; footprint just-40-mark03:1N4148 -> just-40-mark03:1N4148_2
- D2: renamed from D182; footprint just-40-mark03:1N4148 -> just-40-mark03:1N4148_2
- D20: renamed from D200; footprint just-40-mark03:1N4148 -> just-40-mark03:1N4148_2
- D21: renamed from D201; footprint just-40-mark03:1N4148 -> just-40-mark03:1N4148_2
- D22: renamed from D202; footprint just-40-mark03:1N4148 -> just-40-mark03:1N4148_2
- D23: renamed from D203; footprint just-40-mark03:1N4148 -> just-40-mark03:1N4148_2
- D24: renamed from D204; footprint just-40-mark03:1N4148 -> just-40-mark03:1N4148_2
- D25: renamed from D205; footprint just-40-mark03:1N4148 -> just-40-mark03:1N4148_2
- D26: renamed from D206; footprint just-40-mark03:1N4148 -> just-40-mark03:1N4148_2
- D27: renamed from D207; footprint just-40-mark03:1N4148 -> just-40-mark03:1N4148_2
- D28: renamed from D208; footprint just-40-mark03:1N4148 -> just-40-mark03:1N4148_2
- D29: renamed from D209; footprint just-40-mark03:1N4148 -> just-40-mark03:1N4148_2
- D3: renamed from D183; footprint just-40-mark03:1N4148 -> just-40-mark03:1N4148_2
- D30: renamed from D210; footprint just-40-mark03:1N4148 -> just-40-mark03:1N4148_2
- D31: renamed from D211; footprint just-40-mark03:1N4148 -> just-40-mark03:1N4148_2
- D32: renamed from D212; footprint just-40-mark03:1N4148 -> just-40-mark03:1N4148_2
- D33: renamed from D213; footprint just-40-mark03:1N4148 -> just-40-mark03:1N4148_2
- D34: renamed from D214; footprint just-40-mark03:1N4148 -> just-40-mark03:1N4148_2
- D35: renamed from D215; footprint just-40-mark03:1N4148 -> just-40-mark03:1N4148_2
- D36: renamed from D216; footprint just-40-mark03:1N4148 -> just-40-mark03:1N4148_2
- D37: renamed from D217; footprint just-40-mark03:1N4148 -> just-40-mark03:1N4148_2
- D38: renamed from D218; footprint just-40-mark03:1N4148 -> just-40-mark03:1N4148_2
- D39: renamed from D219; footprint just-40-mark03:1N4148 -> just-40-mark03:1N4148_2
- D4: renamed from D184; footprint just-40-mark03:1N4148 -> just-40-mark03:1N4148_2
- D40: renamed from D220; footprint just-40-mark03:1N4148 -> just-40-mark03:1N4148_2
- D5: renamed from D185; footprint just-40-mark03:1N4148 -> just-40-mark03:1N4148_2
- D6: renamed from D186; footprint just-40-mark03:1N4148 -> just-40-mark03:1N4148_2
- D7: renamed from D187; footprint just-40-mark03:1N4148 -> just-40-mark03:1N4148_2
- D8: renamed from D188; footprint just-40-mark03:1N4148 -> just-40-mark03:1N4148_2
- D9: renamed from D189; footprint just-40-mark03:1N4148 -> just-40-mark03:1N4148_2
- H65, H66, H67, H68: footprint just-40-mark03:hole-foot -> just-40-mark03:hole-mount
- H70, H71, H72, H73, H74, H75: footprint just-40-mark03:hole-mount -> just-40-mark03:hole-foot
- SW1: renamed from SW181; footprint just-40-mark03:KS-33-1U_1 -> just-40-mark03:KS-33-1U_2
- SW10: renamed from SW190; footprint just-40-mark03:KS-33-1U_1 -> just-40-mark03:KS-33-1U_2
- SW11: renamed from SW191; footprint just-40-mark03:KS-33-1U_1 -> just-40-mark03:KS-33-1U_2
- SW12: renamed from SW192; footprint just-40-mark03:KS-33-1U_1 -> just-40-mark03:KS-33-1U_2
- SW13: renamed from SW193; footprint just-40-mark03:KS-33-1U_1 -> just-40-mark03:KS-33-1U_2
- SW14: renamed from SW194; footprint just-40-mark03:KS-33-1U_1 -> just-40-mark03:KS-33-1U_2
- SW15: renamed from SW195; footprint just-40-mark03:KS-33-1U_1 -> just-40-mark03:KS-33-1U_2
- SW16: renamed from SW196; footprint just-40-mark03:KS-33-1U_1 -> just-40-mark03:KS-33-1U_2
- SW17: renamed from SW197; footprint just-40-mark03:KS-33-1U_1 -> just-40-mark03:KS-33-1U_2
- SW18: renamed from SW198; footprint just-40-mark03:KS-33-1U_1 -> just-40-mark03:KS-33-1U_2
- SW19: renamed from SW199; footprint just-40-mark03:KS-33-1U_1 -> just-40-mark03:KS-33-1U_2
- SW2: renamed from SW182; footprint just-40-mark03:KS-33-1U_1 -> just-40-mark03:KS-33-1U_2
- SW20: renamed from SW200; footprint just-40-mark03:KS-33-1U_1 -> just-40-mark03:KS-33-1U_2
- SW21: renamed from SW201; footprint just-40-mark03:KS-33-1U_1 -> just-40-mark03:KS-33-1U_2
- SW22: renamed from SW202; footprint just-40-mark03:KS-33-1U_1 -> just-40-mark03:KS-33-1U_2
- SW23: renamed from SW203; footprint just-40-mark03:KS-33-1U_1 -> just-40-mark03:KS-33-1U_2
- SW24: renamed from SW204; footprint just-40-mark03:KS-33-1U_1 -> just-40-mark03:KS-33-1U_2
- SW25: renamed from SW205; footprint just-40-mark03:KS-33-1U_1 -> just-40-mark03:KS-33-1U_2
- SW26: renamed from SW206; footprint just-40-mark03:KS-33-1U_1 -> just-40-mark03:KS-33-1U_2
- SW27: renamed from SW207; footprint just-40-mark03:KS-33-1U_1 -> just-40-mark03:KS-33-1U_2
- SW28: renamed from SW208; footprint just-40-mark03:KS-33-1U_1 -> just-40-mark03:KS-33-1U_2
- SW29: renamed from SW209; footprint just-40-mark03:KS-33-1U_1 -> just-40-mark03:KS-33-1U_2
- SW3: renamed from SW183; footprint just-40-mark03:KS-33-1U_1 -> just-40-mark03:KS-33-1U_2
- SW30: renamed from SW210; footprint just-40-mark03:KS-33-1U_1 -> just-40-mark03:KS-33-1U_2
- SW31: renamed from SW211; footprint just-40-mark03:KS-33-1U_1 -> just-40-mark03:KS-33-1U_2
- SW32: renamed from SW212; footprint just-40-mark03:KS-33-1U_1 -> just-40-mark03:KS-33-1U_2
- SW33: renamed from SW213; footprint just-40-mark03:KS-33-1U_1 -> just-40-mark03:KS-33-1U_2
- SW34: renamed from SW214; footprint just-40-mark03:KS-33-1U_1 -> just-40-mark03:KS-33-1U_2
- SW35: renamed from SW215; footprint just-40-mark03:KS-33-1U_1 -> just-40-mark03:KS-33-1U_2
- SW36: renamed from SW216; footprint just-40-mark03:KS-33-1U_1 -> just-40-mark03:KS-33-1U_2
- SW37: renamed from SW217; footprint just-40-mark03:KS-33-1U_1 -> just-40-mark03:KS-33-1U_2
- SW38: renamed from SW218; footprint just-40-mark03:KS-33-1U_1 -> just-40-mark03:KS-33-1U_2
- SW39: renamed from SW219; footprint just-40-mark03:KS-33-1U_1 -> just-40-mark03:KS-33-1U_2
- SW4: renamed from SW184; footprint just-40-mark03:KS-33-1U_1 -> just-40-mark03:KS-33-1U_2
- SW40: renamed from SW220; footprint just-40-mark03:KS-33-1U_1 -> just-40-mark03:KS-33-1U_2
- SW5: renamed from SW185; footprint just-40-mark03:KS-33-1U_1 -> just-40-mark03:KS-33-1U_2
- SW6: renamed from SW186; footprint just-40-mark03:KS-33-1U_1 -> just-40-mark03:KS-33-1U_2
- SW7: renamed from SW187; footprint just-40-mark03:KS-33-1U_1 -> just-40-mark03:KS-33-1U_2
- SW8: renamed from SW188; footprint just-40-mark03:KS-33-1U_1 -> just-40-mark03:KS-33-1U_2
- SW9: renamed from SW189; footprint just-40-mark03:KS-33-1U_1 -> just-40-mark03:KS-33-1U_2
- moved H2 467.1 mm to (133.0, 29.5)
- moved H3 467.1 mm to (190.0, 29.5)
- moved H1 467.1 mm to (57.0, 29.5)
- moved H4 467.1 mm to (266.0, 29.5)
- moved G*** 459.5 mm to (57.0, 93.0)
- moved H5 451.1 mm to (57.0, 119.5)
- moved H8 451.1 mm to (266.0, 119.5)
- moved H6 451.0 mm to (133.0, 119.5)
- moved H7 451.0 mm to (190.0, 119.5)
- moved D38 450.1 mm to (201.8, 35.2)
- moved SW34 450.0 mm to (104.5, 112.0)
- moved SW35 450.0 mm to (123.5, 112.0)
- moved SW36 450.0 mm to (142.5, 112.0)
- moved SW38 450.0 mm to (180.5, 112.0)
- moved SW39 450.0 mm to (199.5, 112.0)
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- renumbered H57 to H1, H58 to H2, H59 to H3, H60 to H4, H61 to H5, H62 to H6, H63 to H7, H64 to H8
Routing:
- net ROW_80_2: track 0.00 -> 279.4 mm
- net ROW_80_5: track 0.00 -> 254.7 mm
- net COL_801_5: track 0.00 -> 252.5 mm
- net COL_800_5: track 0.00 -> 246.0 mm
- net COL_802_5: track 0.00 -> 236.0 mm
- net COL_801_2: track 0.00 -> 233.7 mm
- net ROW_81_2: track 0.00 -> 230.7 mm
- net COL_800_2: track 0.00 -> 227.2 mm
- net COL_803_5: track 0.00 -> 219.5 mm
- net COL_802_2: track 0.00 -> 217.2 mm
- net ROW_81_5: track 0.00 -> 216.6 mm
- net COL_803_2: track 0.00 -> 200.7 mm
- net COL_804_5: track 0.00 -> 199.6 mm
- net ROW_82_2: track 0.00 -> 186.2 mm
- net COL_804_2: track 0.00 -> 184.3 mm
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- added copper zone on B.Cu, net (none)
- added copper zone on F.Cu, net (none)
- added copper zone on B.Cu, net GND
- added copper zone on F.Cu, net GND
- added copper zone on B.Cu, net GND_2
- added copper zone on F.Cu, net GND_2
- added copper zone on B.Cu, net GND_3
- added copper zone on F.Cu, net GND_3
- added copper zone on B.Cu, net GND_5
- added copper zone on F.Cu, net GND_5
- removed copper zone on B.Cu, net GND_8
- removed copper zone on F.Cu, net GND_8
Other:
- board size 230 x 101.5 mm -> 232 x 642 mm
- board text added: "直 ・ 四 十"
- board text added: "脳"
- board text added: "電"

Commit message: wips
Parts:
- removed A1: RP2350-Zero, just-40-mark03:RP2350-Zero_5
- removed A2, A4: RP2350-Zero, just-40-mark03:RP2350-Tiny-SMD_1
- removed A3: RP2350-Zero, just-40-mark03:RP2350-Tiny-THT_2
- removed the D1 at (61.8, 33.8)
- removed the D10 at (243.8, 35.2)
- removed D100, D101, D102, D103, D104, D105, D106, D107, D108, D109, D110, D111, D112, D113, D114, D115, D116, D117, D118, D119, D120, D41, D42, D43, D44, D45, D46, D47, D48, D49, D50, D51, D52, D53, D54, D55, D56, D57, D58, D59, D60, D61, D62, D63, D64, D65, D66, D67, D68, D69, D70, D71, D72, D73, D74, D75, D76, D77, D78, D79, D80, D81, D82, D83, D84, D85, D86, D87, D88, D89, D90, D91, D92, D93, D94, D95, D96, D97, D98, D99: 1N4148, just-40-mark03:1N4148_2
- removed the D11 at (254.2, 36.8)
- removed the D12 at (261.2, 33.8)
- removed the D13 at (65.2, 35.2)
- removed the D14 at (75.8, 33.8)
- removed the D15 at (89.8, 33.8)
- removed the D16 at (103.8, 33.8)
- removed the D17 at (117.8, 33.8)
- removed the D18 at (194.8, 38.2)
- removed the D19 at (208.8, 38.2)
- removed the D2 at (72.2, 38.2)
- removed the D20 at (222.8, 38.2)
- removed the D21 at (236.8, 38.2)
- removed the D22 at (247.2, 33.8)
- removed the D23 at (257.8, 35.2)
- removed the D24 at (68.8, 36.8)
- removed the D25 at (79.2, 35.2)
- removed the D26 at (93.2, 35.2)
- removed the D27 at (107.2, 35.2)
- removed the D28 at (121.2, 35.2)
- removed the D29 at (198.2, 36.8)
- removed the D3 at (86.2, 38.2)
- removed the D30 at (212.2, 36.8)
- removed the D31 at (226.2, 36.8)
- removed the D32 at (240.2, 36.8)
- removed the D33 at (250.8, 38.2)
- removed the D34 at (82.8, 36.8)
- removed the D35 at (96.8, 36.8)
- removed the D36 at (110.8, 36.8)
- removed the D37 at (124.8, 36.8)
- removed the D38 at (201.8, 35.2)
- removed the D39 at (215.8, 35.2)
- removed the D4 at (100.2, 38.2)
- removed the D40 at (229.8, 35.2)
- removed the D5 at (114.2, 38.2)
- removed the D6 at (128.2, 38.2)
- removed the D7 at (205.2, 33.8)
- removed the D8 at (219.2, 33.8)
- removed the D9 at (233.2, 33.8)
- removed the G*** at (57.0, 93.0)
- removed the G*** at (57.0, 200.5)
- removed the H1 at (57.0, 29.5)
- removed H19, H20, H21, H22, H23, H24, H34, H35, H36, H37, H38, H39, H40, H41, H42, H43, H44, H45, H46, H47, H48, H49, H77, H78, H79, H80, H81, H82, H83, H84: mount-hole, just-40-mark03:hole-mount
- removed the H2 at (133.0, 29.5)
- removed H25, H26, H27, H28, H29, H30, H31, H32, H50, H51, H52, H53, H54, H55, H56, H57, H58, H59, H69, H70, H71, H72, H73, H74, H75, H76: mount-hole, just-40-mark03:hole-foot
- removed the H3 at (190.0, 29.5)
- removed H33: RP2350-Tiny-USB, just-40-mark03:RP2350-Tiny-USB-3
- removed the H4 at (266.0, 29.5)
- removed the H5 at (57.0, 119.5)
- removed the H6 at (133.0, 119.5)
- removed H60, H86: RP2350-Tiny-USB, just-40-mark03:RP2350-Tiny-USB
- removed the H7 at (190.0, 119.5)
- removed the H8 at (266.0, 119.5)
- removed H85: RP2350-Tiny-USB, just-40-mark03:RP2350-Tiny-USB-ref_4
- removed the SW1 at (57.0, 55.0)
- removed the SW10 at (228.0, 55.0)
- removed SW100, SW101, SW102, SW103, SW104, SW105, SW106, SW107, SW108, SW109, SW110, SW111, SW112, SW113, SW114, SW115, SW116, SW117, SW118, SW119, SW120, SW81, SW82, SW83, SW84, SW85, SW86, SW87, SW88, SW89, SW90, SW91, SW92, SW93, SW94, SW95, SW96, SW97, SW98, SW99: ~, just-40-mark03:KS-33-1U_4
- removed the SW11 at (247.0, 55.0)
- removed the SW12 at (266.0, 55.0)
- removed the SW13 at (66.5, 74.0)
- removed the SW14 at (85.5, 74.0)
- removed the SW15 at (104.5, 74.0)
- removed the SW16 at (123.5, 74.0)
- removed the SW17 at (142.5, 74.0)
- removed the SW18 at (161.5, 74.0)
- removed the SW19 at (180.5, 74.0)
- removed the SW2 at (76.0, 55.0)
- removed the SW20 at (199.5, 74.0)
- removed the SW21 at (218.5, 74.0)
- removed the SW22 at (237.5, 74.0)
- removed the SW23 at (256.5, 74.0)
- removed the SW24 at (76.0, 93.0)
- removed the SW25 at (95.0, 93.0)
- removed the SW26 at (114.0, 93.0)
- removed the SW27 at (133.0, 93.0)
- removed the SW28 at (152.0, 93.0)
- removed the SW29 at (171.0, 93.0)
- removed the SW3 at (95.0, 55.0)
- removed the SW30 at (190.0, 93.0)
- removed the SW31 at (209.0, 93.0)
- removed the SW32 at (228.0, 93.0)
- removed the SW33 at (247.0, 93.0)
- removed the SW34 at (104.5, 112.0)
- removed the SW35 at (123.5, 112.0)
- removed the SW36 at (142.5, 112.0)
- removed the SW37 at (161.5, 112.0)
- removed the SW38 at (180.5, 112.0)
- removed the SW39 at (199.5, 112.0)
- removed the SW4 at (114.0, 55.0)
- removed the SW40 at (218.5, 112.0)
- removed SW41, SW42, SW43, SW44, SW45, SW46, SW47, SW48, SW49, SW50, SW51, SW52, SW53, SW54, SW55, SW56, SW57, SW58, SW59, SW60, SW61, SW62, SW63, SW64, SW65, SW66, SW67, SW68, SW69, SW70, SW71, SW72, SW73, SW74, SW75, SW76, SW77, SW78, SW79, SW80: ~, just-40-mark03:KS-33-1U_2
- removed the SW5 at (133.0, 55.0)
- removed the SW6 at (152.0, 55.0)
- removed the SW7 at (171.0, 55.0)
- removed the SW8 at (190.0, 55.0)
- removed the SW9 at (209.0, 55.0)
- added G***: LOGO, just-40-mark03:penguin-sword-40, B.Cu at (237.5, 157.0)
- added U1: ~, just-40-mark03:pro_micro_rp2040_2, F.Cu at (239.5, 81.2)
- H17, H18: footprint just-40-mark03:hole-mount -> just-40-mark03:hole-foot
- moved G*** 477.6 mm to (85.5, 157.0)
- moved D40 475.7 mm to (180.8, 83.5)
- moved D39 475.3 mm to (166.8, 83.5)
- moved D38 474.9 mm to (152.8, 83.5)
- moved D36 474.6 mm to (118.8, 83.5)
- moved D37 474.5 mm to (138.8, 83.5)
- moved D35 474.3 mm to (104.8, 83.5)
- moved D34 474.0 mm to (90.8, 83.5)
- moved D32 458.2 mm to (191.2, 82.0)
- moved D31 457.8 mm to (177.2, 82.0)
- moved D30 457.3 mm to (163.2, 82.0)
- moved D33 457.1 mm to (207.8, 82.0)
- moved D29 457.0 mm to (149.2, 82.0)
- moved D27 456.7 mm to (115.2, 82.0)
- moved D28 456.7 mm to (135.2, 82.0)
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- renumbered D121 to D1, D130 to D10, D131 to D11, D132 to D12, D133 to D13, D134 to D14, D135 to D15, D136 to D16, D137 to D17, D138 to D18, D139 to D19, D122 to D2, D140 to D20, D141 to D21, D142 to D22, D143 to D23, D144 to D24, D145 to D25, D146 to D26, D147 to D27, D148 to D28, D149 to D29, D123 to D3, D150 to D30, D151 to D31, D152 to D32, D153 to D33, D154 to D34, D155 to D35, D156 to D36, D157 to D37, D158 to D38, D159 to D39, D124 to D4, D160 to D40, D125 to D5, D126 to D6, D127 to D7, D128 to D8, D129 to D9, H61 to H1, H62 to H2, H63 to H3, H64 to H4, H65 to H5, H66 to H6, H67 to H7, H68 to H8, SW121 to SW1, SW130 to SW10, SW131 to SW11, SW132 to SW12, SW133 to SW13, SW134 to SW14, SW135 to SW15, SW136 to SW16, SW137 to SW17, SW138 to SW18, SW139 to SW19, SW122 to SW2, SW140 to SW20, SW141 to SW21, SW142 to SW22, SW143 to SW23, SW144 to SW24, SW145 to SW25, SW146 to SW26, SW147 to SW27, SW148 to SW28, SW149 to SW29, SW123 to SW3, SW150 to SW30, SW151 to SW31, SW152 to SW32, SW153 to SW33, SW154 to SW34, SW155 to SW35, SW156 to SW36, SW157 to SW37, SW158 to SW38, SW159 to SW39, SW124 to SW4, SW160 to SW40, SW125 to SW5, SW126 to SW6, SW127 to SW7, SW128 to SW8, SW129 to SW9
Connections:
- net COL_800_5 renamed COL_00
- net COL_801_5 renamed COL_01
- net COL_802_5 renamed COL_02
- net COL_803_5 renamed COL_03
- net COL_804_5 renamed COL_04
- net COL_805_5 renamed COL_05
- net COL_806_5 renamed COL_06
- net COL_807_5 renamed COL_07
- net COL_808_5 renamed COL_08
- net COL_809_5 renamed COL_09
- net COL_810_5 renamed COL_10
- net ROW_80_5 renamed ROW_0
- net ROW_81_5 renamed ROW_1
- net ROW_82_5 renamed ROW_2
- net ROW_83_5 renamed ROW_3
- SW12 pad 1: COL_811_5 -> COL_11
Routing:
- net ROW_80_2: track 279.4 -> 0.00 mm
- net COL_801_2: track 233.7 -> 0.00 mm
- net ROW_81_2: track 230.7 -> 0.00 mm
- net COL_800_2: track 227.2 -> 0.00 mm
- net COL_802_2: track 217.2 -> 0.00 mm
- net ROW_80: track 209.1 -> 0.00 mm, vias 1 -> 0
- net ROW_81: track 205.5 -> 0.00 mm, vias 1 -> 0
- net COL_803_2: track 200.7 -> 0.00 mm
- net ROW_82: track 192.0 -> 0.00 mm, vias 1 -> 0
- net ROW_82_2: track 186.2 -> 0.00 mm
- net COL_804_2: track 184.3 -> 0.00 mm
- net COL_801: track 171.3 -> 0.00 mm, vias 2 -> 0
- net COL_800: track 171.3 -> 0.00 mm, vias 2 -> 0
- net COL_805_2: track 167.8 -> 0.00 mm
- net ROW_83: track 154.0 -> 0.00 mm, vias 1 -> 0
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- removed copper zone on B.Cu, net (none)
- removed copper zone on F.Cu, net (none)
- removed copper zone on B.Cu, net GND_2
- removed copper zone on F.Cu, net GND_2
- removed copper zone on B.Cu, net GND_3
- removed copper zone on F.Cu, net GND_3
- removed copper zone on B.Cu, net GND_5
- removed copper zone on F.Cu, net GND_5
Other:
- board size 232 x 642 mm -> 232 x 96.5 mm
- board text removed: "Just 40"
- board text removed: "脳"
- board text removed: "電"
