File: kicad/just-40-mark03/just-40-mark03.kicad_pcb (KiCad board)
At the start: 2 copper layers, 232 x 96.5 mm, 101 parts

Commit message: done: mark03
Parts:
- removed G*** (x2): LOGO, just-40-mark03:penguin-sword-40
- removed U1: ~, just-40-mark03:pro_micro_rp2040_2
- added A1: RP2350-Tiny, just-40-mark03:RP2350-Tiny-SMD, F.Cu at (57.0, 399.0)
- added H19: mount-hole, just-40-mark03:hole-foot, F.Cu at (199.5, 389.5)
- D1, D10, D11, D12, D13, D14, D15, D16, D17, D18, D19, D2, D20, D21, D22, D23, D24, D25, D26, D27, D28, D29, D3, D30, D31, D32, D33, D34, D35, D36, D37, D38, D39, D4, D40, D5, D6, D7, D8, D9: footprint just-40-mark03:1N4148_2 -> just-40-mark03:1N4148_3
- H9: value mount-hole -> RP2350-Tiny-USB; footprint just-40-mark03:hole-foot -> just-40-mark03:RP2350-Tiny-USB-3
- SW1, SW10, SW11, SW12, SW13, SW14, SW15, SW16, SW17, SW18, SW19, SW2, SW20, SW21, SW22, SW23, SW24, SW25, SW26, SW27, SW28, SW29, SW3, SW30, SW31, SW32, SW33, SW34, SW35, SW36, SW37, SW38, SW39, SW4, SW40, SW5, SW6, SW7, SW8, SW9: footprint just-40-mark03:KS-33-1U_4 -> just-40-mark03:KS-33v3-1U_4
- moved H14 339.4 mm to (53.0, 422.0)
- moved D39 337.0 mm to (207.8, 418.0)
- moved D36 336.0 mm to (150.8, 418.0)
- moved D40 335.8 mm to (210.2, 418.0)
- moved D34 335.2 mm to (112.8, 418.0)
- moved D38 335.1 mm to (172.2, 418.0)
- moved D37 334.8 mm to (153.2, 418.0)
- moved D35 334.7 mm to (115.2, 418.0)
- moved H15 331.5 mm to (133.0, 418.0)
- moved H17 329.6 mm to (270.0, 422.0)
- moved H18 328.0 mm to (123.5, 389.5)
- moved H16 324.9 mm to (190.0, 418.0)
- moved D33 318.5 mm to (238.8, 399.0)
- moved D32 318.3 mm to (219.8, 399.0)
- moved D31 317.9 mm to (200.8, 399.0)
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Connections:
- net ROW_0 renamed ROW_0_2
- net ROW_1 renamed ROW_1_2
- net ROW_2 renamed ROW_2_2
- net ROW_3 renamed ROW_3_2
- SW1 pad 1: COL_00 -> COL_00_2
- SW10 pad 1: COL_09 -> COL_09_2
- SW11 pad 1: COL_10 -> COL_10_2
- SW12 pad 1: COL_11 -> COL_11_2
- SW13 pad 1: COL_00 -> COL_01_2
- SW14 pad 1: COL_01 -> COL_02_2
- SW15 pad 1: COL_02 -> COL_03_2
- SW16 pad 1: COL_03 -> COL_04_2
- SW17 pad 1: COL_04 -> COL_05_2
- SW18 pad 1: COL_05 -> COL_06_2
- SW19 pad 1: COL_06 -> COL_07_2
- SW2 pad 1: COL_01 -> COL_01_2
- SW20 pad 1: COL_07 -> COL_08_2
- SW21 pad 1: COL_08 -> COL_09_2
- SW22 pad 1: COL_09 -> COL_10_2
- SW23 pad 1: COL_10 -> COL_11_2
- SW24 pad 1: COL_00 -> COL_02_2
- SW25 pad 1: COL_01 -> COL_03_2
- SW26 pad 1: COL_02 -> COL_04_2
- SW27 pad 1: COL_03 -> COL_05_2
- SW28 pad 1: COL_04 -> COL_06_2
- SW29 pad 1: COL_05 -> COL_07_2
- SW3 pad 1: COL_02 -> COL_02_2
- SW30 pad 1: COL_06 -> COL_08_2
- SW31 pad 1: COL_07 -> COL_09_2
- SW32 pad 1: COL_08 -> COL_10_2
- SW33 pad 1: COL_09 -> COL_11_2
- SW34 pad 1: COL_01 -> COL_04_2
- SW35 pad 1: COL_02 -> COL_05_2
- SW36 pad 1: COL_03 -> COL_06_2
- SW37 pad 1: COL_04 -> COL_07_2
- SW38 pad 1: COL_05 -> COL_08_2
- SW39 pad 1: COL_06 -> COL_09_2
- SW4 pad 1: COL_03 -> COL_03_2
- SW40 pad 1: COL_07 -> COL_10_2
- SW5 pad 1: COL_04 -> COL_04_2
- SW6 pad 1: COL_05 -> COL_05_2
- SW7 pad 1: COL_06 -> COL_06_2
- SW8 pad 1: COL_07 -> COL_07_2
- SW9 pad 1: COL_08 -> COL_08_2
Routing:
- net COL_01: track 260.6 -> 0.00 mm, vias 2 -> 0
- net COL_00: track 257.1 -> 0.00 mm, vias 2 -> 0
- net COL_10_2: track 0.00 -> 252.0 mm
- net COL_11_2: track 0.00 -> 250.9 mm
- net COL_02: track 241.9 -> 0.00 mm, vias 2 -> 0
- net COL_09_2: track 0.00 -> 230.1 mm
- net COL_03: track 223.2 -> 0.00 mm, vias 2 -> 0
- net COL_08_2: track 0.00 -> 208.3 mm
- net COL_05: track 195.1 -> 0.00 mm, vias 3 -> 0
- net COL_07_2: track 0.00 -> 185.4 mm
- net COL_04: track 182.7 -> 0.00 mm, vias 2 -> 0
- net COL_06: track 173.1 -> 0.00 mm, vias 3 -> 0
- net COL_06_2: track 0.00 -> 161.8 mm
- net COL_07: track 151.1 -> 0.00 mm, vias 3 -> 0
- net COL_05_2: track 0.00 -> 143.5 mm
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- added copper zone on B.Cu, net GND_2
- added copper zone on F.Cu, net GND_2
- removed copper zone on B.Cu, net GND
- removed copper zone on F.Cu, net GND
Other:
- board size 232 x 96.5 mm -> 230 x 79 mm
