File: kicad/just-40-mark03/just-40-mark03.kicad_sch (KiCad schematic)
At the start: 102 parts

Commit message: mark03
Parts:
- removed A1: RP2350-Zero, just-40-mark03:RP2350-Tiny-SMD, symbol just-40-mark03:RP2350-Zero
- removed A2, A3, A4, A5, A6, A7: neopixel, just-40-mark03:SK6812MINI-E, symbol just-40-mark03:SK6812MINI-E
- removed D1, D10, D11, D12, D13, D14, D15, D16, D17, D18, D19, D2, D20, D21, D22, D23, D24, D25, D26, D27, D28, D29, D3, D30, D31, D32, D33, D34, D35, D36, D37, D38, D39, D4, D40, D5, D6, D7, D8, D9: 1N4148, just-40-mark03:1N4148, symbol just-40-mark03:1N4148
- removed H1, H2, H3, H4, H5, H6, H7, H8: mount-hole, just-40-mark03:hole-mount, symbol just-40-hhkb:mount-hole
- removed H10, H11, H12, H13, H9: mount-hole, just-40-mark03:hole-foot, symbol just-40-hhkb:mount-hole
- removed H14: RP2350-Tiny-USB, just-40-mark03:RP2350-Tiny-USB-4, symbol just-40:RP2350-Tiny-USB
- removed R1: R, just-40-mark03:330_ohm, symbol Device:R
- removed SW1, SW10, SW11, SW12, SW13, SW14, SW15, SW16, SW17, SW18, SW19, SW2, SW20, SW21, SW22, SW23, SW24, SW25, SW26, SW27, SW28, SW29, SW3, SW30, SW31, SW32, SW33, SW34, SW35, SW36, SW37, SW38, SW39, SW4, SW40, SW5, SW6, SW7, SW8, SW9: ~, just-40-mark03:KS-33-1U, symbol just-40-mark03:KS-33
- added A27: RP2350-Zero, just-40-mark03:RP2350-Zero_1, symbol just-40-mark03:RP2350-Zero
- added D181, D182, D183, D184, D185, D186, D187, D188, D189, D190, D191, D192, D193, D194, D195, D196, D197, D198, D199, D200, D201, D202, D203, D204, D205, D206, D207, D208, D209, D210, D211, D212, D213, D214, D215, D216, D217, D218, D219, D220: 1N4148, just-40-mark03:1N4148, symbol just-40-mark03:1N4148
- added H57, H58, H59, H60, H61, H62, H63, H64, H70, H71, H72, H73, H74, H75: mount-hole, just-40-mark03:hole-mount, symbol just-40-hhkb:mount-hole
- added H65, H66, H67, H68, H69: mount-hole, just-40-mark03:hole-foot, symbol just-40-hhkb:mount-hole
- added SW181, SW182, SW183, SW184, SW185, SW186, SW187, SW188, SW189, SW190, SW191, SW192, SW193, SW194, SW195, SW196, SW197, SW198, SW199, SW200, SW201, SW202, SW203, SW204, SW205, SW206, SW207, SW208, SW209, SW210, SW211, SW212, SW213, SW214, SW215, SW216, SW217, SW218, SW219, SW220: (no value), just-40-mark03:KS-33-1U_1, symbol just-40-mark03:KS-33
Connections:
- new net: D181.A, SW181.2 (B)
- new net: D203.A, SW203.2 (B)
- new net: D201.A, SW201.2 (B)
- new net: D215.A, SW215.2 (B)
- new net: D186.A, SW186.2 (B)
- new net: D209.A, SW209.2 (B)
- new net: D192.A, SW192.2 (B)
- new net: D198.A, SW198.2 (B)
- new net: D187.A, SW187.2 (B)
- new net: D205.A, SW205.2 (B)
- new net: D197.A, SW197.2 (B)
- new net: D204.A, SW204.2 (B)
- new net: D207.A, SW207.2 (B)
- new net: D184.A, SW184.2 (B)
- new net: D193.A, SW193.2 (B)
- new net: D190.A, SW190.2 (B)
- new net: D206.A, SW206.2 (B)
- new net: D185.A, SW185.2 (B)
- new net: D191.A, SW191.2 (B)
- new net: D199.A, SW199.2 (B)
- new net: D212.A, SW212.2 (B)
- new net: D218.A, SW218.2 (B)
- new net: D202.A, SW202.2 (B)
- new net: D194.A, SW194.2 (B)
- new net: D219.A, SW219.2 (B)
- new net: D220.A, SW220.2 (B)
- new net: D213.A, SW213.2 (B)
- new net: D183.A, SW183.2 (B)
- new net: D217.A, SW217.2 (B)
- new net: D211.A, SW211.2 (B)
- new net: D210.A, SW210.2 (B)
- new net: D188.A, SW188.2 (B)
- new net: D189.A, SW189.2 (B)
- new net: D195.A, SW195.2 (B)
- new net: D196.A, SW196.2 (B)
- new net: D214.A, SW214.2 (B)
- new net: D182.A, SW182.2 (B)
- new net: D208.A, SW208.2 (B)
- new net: D216.A, SW216.2 (B)
- new net: D200.A, SW200.2 (B)
- new net COL_800: A27.27 (GPIO27_ADC1), SW181.1 (A), SW193.1 (A), SW204.1 (A)
- new net COL_801: A27.26 (GPIO26_ADC0), SW182.1 (A), SW194.1 (A), SW205.1 (A), SW214.1 (A)
- new net COL_802: A27.15 (GPIO15), SW183.1 (A), SW195.1 (A), SW206.1 (A), SW215.1 (A)
- new net COL_803: A27.14 (GPIO14), SW184.1 (A), SW196.1 (A), SW207.1 (A), SW216.1 (A)
- new net COL_804: A27.13 (GPIO13), SW185.1 (A), SW197.1 (A), SW208.1 (A), SW217.1 (A)
- new net COL_805: A27.12 (GPIO12), SW186.1 (A), SW198.1 (A), SW209.1 (A), SW218.1 (A)
- new net COL_806: A27.10 (GPIO10), SW187.1 (A), SW199.1 (A), SW210.1 (A), SW219.1 (A)
- new net COL_807: A27.9 (GPIO9), SW188.1 (A), SW200.1 (A), SW211.1 (A), SW220.1 (A)
- new net COL_808: A27.8 (GPIO8), SW189.1 (A), SW201.1 (A), SW212.1 (A)
- new net COL_809: A27.7 (GPIO7), SW190.1 (A), SW202.1 (A), SW213.1 (A)
- new net COL_810: A27.6 (GPIO6), SW191.1 (A), SW203.1 (A)
- new net COL_811: A27.5 (GPIO5), SW192.1 (A)
- new net GND_8: A27.GND
- new net ROW_80: A27.1 (GPIO1), D181.K, D182.K, D183.K, D184.K, D185.K, D186.K, D187.K, D188.K, D189.K, D190.K, D191.K, D192.K
- new net ROW_81: A27.2 (GPIO2), D193.K, D194.K, D195.K, D196.K, D197.K, D198.K, D199.K, D200.K, D201.K, D202.K, D203.K
- new net ROW_82: A27.29 (GPIO29_ADC2), D204.K, D205.K, D206.K, D207.K, D208.K, D209.K, D210.K, D211.K, D212.K, D213.K
- new net ROW_83: A27.28 (GPIO28_ADC2), D214.K, D215.K, D216.K, D217.K, D218.K, D219.K, D220.K
- no-connect marks 5 -> 6
