File: kicad/just-40-mark03/just-40-mark03.kicad_sch (KiCad schematic)
At the start: 410 parts

Commit message: wips
Parts:
- removed A1: RP2350-Zero, just-40-mark03:RP2350-Zero_5, symbol just-40-mark03:RP2350-Zero
- removed A2, A4: RP2350-Zero, just-40-mark03:RP2350-Tiny-SMD_1, symbol just-40-mark03:RP2350-Zero
- removed A3: RP2350-Zero, just-40-mark03:RP2350-Tiny-THT_2, symbol just-40-mark03:RP2350-Zero
- removed D1, D10, D100, D101, D102, D103, D104, D105, D106, D107, D108, D109, D11, D110, D111, D112, D113, D114, D115, D116, D117, D118, D119, D12, D120, D13, D14, D15, D16, D17, D18, D19, D2, D20, D21, D22, D23, D24, D25, D26, D27, D28, D29, D3, D30, D31, D32, D33, D34, D35, D36, D37, D38, D39, D4, D40, D41, D42, D43, D44, D45, D46, D47, D48, D49, D5, D50, D51, D52, D53, D54, D55, D56, D57, D58, D59, D6, D60, D61, D62, D63, D64, D65, D66, D67, D68, D69, D7, D70, D71, D72, D73, D74, D75, D76, D77, D78, D79, D8, D80, D81, D82, D83, D84, D85, D86, D87, D88, D89, D9, D90, D91, D92, D93, D94, D95, D96, D97, D98, D99: 1N4148, just-40-mark03:1N4148_2, symbol just-40-mark03:1N4148
- removed H1, H19, H2, H20, H21, H22, H23, H24, H3, H34, H35, H36, H37, H38, H39, H4, H40, H41, H42, H43, H44, H45, H46, H47, H48, H49, H5, H6, H7, H77, H78, H79, H8, H80, H81, H82, H83, H84: mount-hole, just-40-mark03:hole-mount, symbol just-40-hhkb:mount-hole
- removed H25, H26, H27, H28, H29, H30, H31, H32, H50, H51, H52, H53, H54, H55, H56, H57, H58, H59, H69, H70, H71, H72, H73, H74, H75, H76: mount-hole, just-40-mark03:hole-foot, symbol just-40-hhkb:mount-hole
- removed H33: RP2350-Tiny-USB, just-40-mark03:RP2350-Tiny-USB-3, symbol just-40-mark03:RP2350-Tiny-USB
- removed H60, H86: RP2350-Tiny-USB, just-40-mark03:RP2350-Tiny-USB, symbol just-40-mark03:RP2350-Tiny-USB
- removed H85: RP2350-Tiny-USB, just-40-mark03:RP2350-Tiny-USB-ref_4, symbol just-40-mark03:RP2350-Tiny-USB
- removed SW1, SW10, SW11, SW12, SW13, SW14, SW15, SW16, SW17, SW18, SW19, SW2, SW20, SW21, SW22, SW23, SW24, SW25, SW26, SW27, SW28, SW29, SW3, SW30, SW31, SW32, SW33, SW34, SW35, SW36, SW37, SW38, SW39, SW4, SW40, SW41, SW42, SW43, SW44, SW45, SW46, SW47, SW48, SW49, SW5, SW50, SW51, SW52, SW53, SW54, SW55, SW56, SW57, SW58, SW59, SW6, SW60, SW61, SW62, SW63, SW64, SW65, SW66, SW67, SW68, SW69, SW7, SW70, SW71, SW72, SW73, SW74, SW75, SW76, SW77, SW78, SW79, SW8, SW80, SW9: (no value), just-40-mark03:KS-33-1U_2, symbol just-40-mark03:KS-33
- removed SW100, SW101, SW102, SW103, SW104, SW105, SW106, SW107, SW108, SW109, SW110, SW111, SW112, SW113, SW114, SW115, SW116, SW117, SW118, SW119, SW120, SW81, SW82, SW83, SW84, SW85, SW86, SW87, SW88, SW89, SW90, SW91, SW92, SW93, SW94, SW95, SW96, SW97, SW98, SW99: (no value), just-40-mark03:KS-33-1U_4, symbol just-40-mark03:KS-33
- added U1: (no value), just-40-mark03:pro_micro_rp2040_2, symbol base:pro_micro_rp2040
- H17, H18: footprint just-40-mark03:hole-mount -> just-40-mark03:hole-foot
- renumbered D121 to D1, D130 to D10, D131 to D11, D132 to D12, D133 to D13, D134 to D14, D135 to D15, D136 to D16, D137 to D17, D138 to D18, D139 to D19, D122 to D2, D140 to D20, D141 to D21, D142 to D22, D143 to D23, D144 to D24, D145 to D25, D146 to D26, D147 to D27, D148 to D28, D149 to D29, D123 to D3, D150 to D30, D151 to D31, D152 to D32, D153 to D33, D154 to D34, D155 to D35, D156 to D36, D157 to D37, D158 to D38, D159 to D39, D124 to D4, D160 to D40, D125 to D5, D126 to D6, D127 to D7, D128 to D8, D129 to D9, H61 to H1, H62 to H2, H63 to H3, H64 to H4, H65 to H5, H66 to H6, H67 to H7, H68 to H8, SW121 to SW1, SW130 to SW10, SW131 to SW11, SW132 to SW12, SW133 to SW13, SW134 to SW14, SW135 to SW15, SW136 to SW16, SW137 to SW17, SW138 to SW18, SW139 to SW19, SW122 to SW2, SW140 to SW20, SW141 to SW21, SW142 to SW22, SW143 to SW23, SW144 to SW24, SW145 to SW25, SW146 to SW26, SW147 to SW27, SW148 to SW28, SW149 to SW29, SW123 to SW3, SW150 to SW30, SW151 to SW31, SW152 to SW32, SW153 to SW33, SW154 to SW34, SW155 to SW35, SW156 to SW36, SW157 to SW37, SW158 to SW38, SW159 to SW39, SW124 to SW4, SW160 to SW40, SW125 to SW5, SW126 to SW6, SW127 to SW7, SW128 to SW8, SW129 to SW9
Connections:
- net GND: now also U1.GND
- net COL_800_5 renamed COL_00
- net COL_00: now also U1.27 (GP27)
- net COL_801_5 renamed COL_01
- net COL_01: now also U1.26 (GP26)
- net COL_802_5 renamed COL_02
- net COL_02: now also U1.22 (GP22)
- net COL_803_5 renamed COL_03
- net COL_03: now also U1.20 (GP20)
- net COL_804_5 renamed COL_04
- net COL_04: now also U1.21 (GP21)
- net COL_805_5 renamed COL_05
- net COL_05: now also U1.2 (GP2)
- net COL_806_5 renamed COL_06
- net COL_06: now also U1.3 (GP3)
- net COL_807_5 renamed COL_07
- net COL_07: now also U1.4 (GP4)
- net COL_808_5 renamed COL_08
- net COL_08: now also U1.5 (GP5)
- net COL_809_5 renamed COL_09
- net COL_09: now also U1.23 (GP23)
- net COL_810_5 renamed COL_10
- net COL_10: now also U1.28 (GP28)
- net COL_811_5 renamed COL_11
- net COL_11: now also U1.29 (GP29)
- net ROW_80_5 renamed ROW_0
- net ROW_0: now also U1.9 (GP9)
- net ROW_81_5 renamed ROW_1
- net ROW_1: now also U1.8 (GP8)
- net ROW_82_5 renamed ROW_2
- net ROW_2: now also U1.7 (GP7)
- net ROW_83_5 renamed ROW_3
- net ROW_3: now also U1.6 (GP6)
Other:
- moved on the sheet: D1, D10, D11, D12, D13, D14, D15, D16, D17, D18, D19, D2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
