File: kicad/just-40-mark03/just-40-mark03.kicad_sch (KiCad schematic)
At the start: 99 parts

Commit message: done: mark03
Parts:
- removed H1, H2, H3, H4, H5, H6, H7, H8: mount-hole, just-40-mark03:hole-mount, symbol just-40-hhkb:mount-hole
- removed H10, H11, H12, H13, H14, H15, H16, H17, H18, H9: mount-hole, just-40-mark03:hole-foot, symbol just-40-hhkb:mount-hole
- removed U1: (no value), just-40-mark03:pro_micro_rp2040_2, symbol base:pro_micro_rp2040
- added A1: RP2350-Tiny, just-40-mark03:RP2350-Tiny-SMD, symbol just-40-mark03:RP2350-Tiny
- added H1, H2, H3, H4, H5, H6, H7, H8: mount-hole, just-40-mark03:hole-mount, symbol just-40-mark03:mount-hole
- added H10, H11, H12, H13, H14, H15, H16, H17, H18, H19: mount-hole, just-40-mark03:hole-foot, symbol just-40-mark03:mount-hole
- added H9: RP2350-Tiny-USB, just-40-mark03:RP2350-Tiny-USB-3, symbol just-40-mark03:RP2350-Tiny-USB
- D1, D10, D11, D12, D13, D14, D15, D16, D17, D18, D19, D2, D20, D21, D22, D23, D24, D25, D26, D27, D28, D29, D3, D30, D31, D32, D33, D34, D35, D36, D37, D38, D39, D4, D40, D5, D6, D7, D8, D9: footprint just-40-mark03:1N4148_2 -> just-40-mark03:1N4148_3
- SW1, SW10, SW11, SW12, SW13, SW14, SW15, SW16, SW17, SW18, SW19, SW2, SW20, SW21, SW22, SW23, SW24, SW25, SW26, SW27, SW28, SW29, SW3, SW30, SW31, SW32, SW33, SW34, SW35, SW36, SW37, SW38, SW39, SW4, SW40, SW5, SW6, SW7, SW8, SW9: footprint just-40-mark03:KS-33-1U_4 -> just-40-mark03:KS-33v3-1U_4
Connections:
- removed net COL_00: SW1.1 (A), SW13.1 (A), SW24.1 (A)
- removed net COL_01: SW14.1 (A), SW2.1 (A), SW25.1 (A), SW34.1 (A)
- removed net COL_02: SW15.1 (A), SW26.1 (A), SW3.1 (A), SW35.1 (A)
- removed net COL_03: SW16.1 (A), SW27.1 (A), SW36.1 (A), SW4.1 (A)
- removed net COL_04: SW17.1 (A), SW28.1 (A), SW37.1 (A), SW5.1 (A)
- removed net COL_05: SW18.1 (A), SW29.1 (A), SW38.1 (A), SW6.1 (A)
- removed net COL_06: SW19.1 (A), SW30.1 (A), SW39.1 (A), SW7.1 (A)
- removed net COL_07: SW20.1 (A), SW31.1 (A), SW40.1 (A), SW8.1 (A)
- removed net COL_08: SW21.1 (A), SW32.1 (A), SW9.1 (A)
- removed net COL_09: SW10.1 (A), SW22.1 (A), SW33.1 (A)
- net COL_10 renamed COL_10_2
- net COL_10_2: now also SW22.1 (A), SW32.1 (A), SW40.1 (A), A1.10 (GPIO10); no longer SW23.1 (A)
- net COL_11 renamed COL_11_2
- net COL_11_2: now also SW23.1 (A), SW33.1 (A), A1.9 (GPIO9)
- net ROW_0 renamed ROW_0_2
- net ROW_0_2: now also A1.0 (GPIO0)
- net ROW_1 renamed ROW_1_2
- net ROW_1_2: now also A1.3 (GPIO3)
- net ROW_2 renamed ROW_2_2
- net ROW_2_2: now also A1.28 (GPIO28_ADC2)
- net ROW_3 renamed ROW_3_2
- net ROW_3_2: now also A1.8 (GPIO8)
- new net COL_00_2: A1.1 (GPIO1), SW1.1 (A)
- new net COL_01_2: A1.2 (GPIO2), SW13.1 (A), SW2.1 (A)
- new net COL_02_2: A1.29 (GPIO29_ADC2), SW14.1 (A), SW24.1 (A), SW3.1 (A)
- new net COL_03_2: A1.27 (GPIO27_ADC1), SW15.1 (A), SW25.1 (A), SW4.1 (A)
- new net COL_04_2: A1.26 (GPIO26_ADC0), SW16.1 (A), SW26.1 (A), SW34.1 (A), SW5.1 (A)
- new net COL_05_2: A1.15 (GPIO15), SW17.1 (A), SW27.1 (A), SW35.1 (A), SW6.1 (A)
- new net COL_06_2: A1.14 (GPIO14), SW18.1 (A), SW28.1 (A), SW36.1 (A), SW7.1 (A)
- new net COL_07_2: A1.13 (GPIO13), SW19.1 (A), SW29.1 (A), SW37.1 (A), SW8.1 (A)
- new net COL_08_2: A1.12 (GPIO12), SW20.1 (A), SW30.1 (A), SW38.1 (A), SW9.1 (A)
- new net COL_09_2: A1.11 (GPIO11), SW10.1 (A), SW21.1 (A), SW31.1 (A), SW39.1 (A)
- new net GND_2: A1.GND
- no-connect marks 0 -> 2
